File: pcb/v1/speedometer.kicad_sch (KiCad schematic)
At the start: 4 parts, among them U4 4511, U5 4511, U6 4511

Commit message: end v1, move to modular design
Parts:
- added Q1, Q10, Q11, Q12, Q13, Q14, Q2, Q3, Q4: BSS138, Package_TO_SOT_SMD:SOT-23, symbol Transistor_FET:BSS138
- added R10, R11, R12, R13, R14, R6, R7, R8, R9: 1k 1/10W +-1%, Resistor_SMD:R_0603_1608Metric, symbol Device:R_Small
- added RN1, RN10, RN11, RN12, RN2, RN26, RN27, RN28, RN29, RN3, RN30, RN31, RN4, RN5, RN6, RN7, RN8, RN9: 560Ω ±5% 63mW, Resistor_SMD:R_Array_Convex_4x0603, symbol Device:R_Pack04
- added U1, U2, U29, U3, U30, U31, U7, U8, U9: KCSC02-123, Display_7Segment:KCSC02-123, symbol Display_Character:KCSC02-123
- added U10, U14, U15, U19, U20, U21: HDSP-7801, Display_7Segment:HDSP-7801, symbol Display_Character:HDSP-7801
- added U11, U12, U13, U16, U17, U18: 4511, Package_SO:TSSOP-16_4.4x5mm_P0.65mm, symbol 4xxx_IEEE:4511
- added U24, U25, U26: HDSP-7801, DashDash:SA15-11xxx, symbol Display_Character:HDSP-7801
- added U40, U41, U42, U43, U44, U45, U46: 74HC595, Package_SO:TSSOP-16_4.4x5mm_P0.65mm, symbol 74xx:74HC595
- U4, U5, U6: footprint Package_SO:SOP-16_4.55x10.3mm_P1.27mm -> Package_SO:TSSOP-16_4.4x5mm_P0.65mm
Connections:
- net +12V: now also U11.16 (Vdd), U12.16 (Vdd), U13.16 (Vdd), U16.16 (Vdd), U17.16 (Vdd), U18.16 (Vdd), U40.16 (VCC), U41.16 (VCC), U42.16 (VCC), U43.16 (VCC), U44.16 (VCC), U45.16 (VCC), U46.16 (VCC)
- net GND: now also U4.5 (~{EL}), U5.5 (~{EL}), U6.5 (~{EL}), Q1.2 (S), Q10.2 (S), Q11.2 (S), Q12.2 (S), Q13.2 (S), Q14.2 (S), Q2.2 (S), Q3.2 (S), Q4.2 (S), RN10.8 (R1.2), U11.5 (~{EL}), U11.8 (Vss), U12.5 (~{EL}), U12.8 (Vss), U13.5 (~{EL}), U13.8 (Vss), U16.5 (~{EL}), U16.8 (Vss), U17.5 (~{EL}), U17.8 (Vss), U18.5 (~{EL}), U18.8 (Vss), U40.8 (GND), U41.8 (GND), U42.8 (GND), U43.8 (GND), U44.8 (GND), U45.8 (GND), U46.8 (GND)
- net S_7S_A_DB: now reaches U4.1 (DB)
- net S_7S_A_DB: now also U44.5 (QF)
- net at U4.10 (Qd): now also RN26.8 (R1.2)
- net at U4.11 (Qc): now also RN26.7 (R2.2)
- net at U4.12 (Qb): now also RN26.6 (R3.2)
- net at U4.13 (Qa): now also RN26.5 (R4.2)
- net at U4.14 (Qg): now also RN27.7 (R2.2)
- net at U4.15 (Qf): now also RN27.6 (R3.2)
- net S_7S_A_DC: now reaches U4.2 (DC)
- net S_7S_A_DC: now also U44.6 (QG)
- net S_7S_A_LT: now reaches U4.3 (~{LT})
- net S_7S_A_LT: now also U45.15 (QA)
- net S_7S_A_BI: now reaches U4.4 (~{BI})
- net S_7S_A_BI: now also U45.1 (QB)
- net S_7S_A_DD: now reaches U4.6 (DD)
- net S_7S_A_DD: now also U44.7 (QH)
- net S_7S_A_DA: now reaches U4.7 (DA)
- net S_7S_A_DA: now also U44.4 (QE)
- net at U4.9 (Qe): now also RN27.5 (R4.2)
- net S_7S_B_DB: now reaches U6.1 (DB)
- net S_7S_B_DB: now also U5.1 (DB), U45.3 (QD), U46.1 (QB)
- net at U6.10 (Qd): now also RN30.8 (R1.2)
- net at U6.11 (Qc): now also RN30.7 (R2.2)
- net at U6.12 (Qb): now also RN30.6 (R3.2)
- net at U6.13 (Qa): now also RN30.5 (R4.2)
- net at U6.14 (Qg): now also RN31.7 (R2.2)
- net at U6.15 (Qf): now also RN31.6 (R3.2)
- net S_7S_B_DC: now reaches U6.2 (DC)
- net S_7S_B_DC: now also U5.2 (DC), U45.4 (QE), U46.2 (QC)
- net S_7S_B_LT: now reaches U6.3 (~{LT})
- net S_7S_B_LT: now also U5.3 (~{LT}), U45.6 (QG), U46.4 (QE)
- net S_7S_B_BI: now reaches U6.4 (~{BI})
- net S_7S_B_BI: now also U5.4 (~{BI}), U45.7 (QH), U46.5 (QF)
- net S_7S_B_DD: now reaches U6.6 (DD)
- net S_7S_B_DD: now also U5.6 (DD), U45.5 (QF), U46.3 (QD)
- net S_7S_B_DA: now reaches U6.7 (DA)
- net S_7S_B_DA: now also U5.7 (DA), U45.2 (QC), U46.15 (QA)
- net at U6.9 (Qe): now also RN31.5 (R4.2)
- net at U5.10 (Qd): now also RN28.8 (R1.2)
- net at U5.11 (Qc): now also RN28.7 (R2.2)
- net at U5.12 (Qb): now also RN28.6 (R3.2)
- net at U5.13 (Qa): now also RN28.5 (R4.2)
- net at U5.14 (Qg): now also RN29.7 (R2.2)
- net at U5.15 (Qf): now also RN29.6 (R3.2)
- net at U5.9 (Qe): now also RN29.5 (R4.2)
- new net: Q12.1 (G), R12.2
- new net: Q12.3 (D), U26.1 (CA), U26.6 (CA)
- new net: Q14.1 (G), R14.2
- new net: Q14.3 (D), U15.1 (CA), U15.6 (CA)
- new net: RN7.1 (R1.1), U19.5 (D)
- new net: RN7.2 (R2.1), U19.8 (C)
- new net: RN7.3 (R3.1), U19.9 (B)
- new net: RN7.4 (R4.1), U19.10 (A)
- new net: RN7.5 (R4.2), U16.13 (Qa)
- new net: RN7.6 (R3.2), U16.12 (Qb)
- new net: RN7.7 (R2.2), U16.11 (Qc)
- new net: RN7.8 (R1.2), U16.10 (Qd)
- new net: RN31.1 (R1.1), U26.7 (DP)
- new net: RN31.2 (R2.1), U26.3 (G)
- new net: RN31.3 (R3.1), U26.2 (F)
- new net: RN31.4 (R4.1), U26.4 (E)
- new net: RN9.1 (R1.1), U20.5 (D)
- new net: RN9.2 (R2.1), U20.8 (C)
- new net: RN9.3 (R3.1), U20.9 (B)
- new net: RN9.4 (R4.1), U20.10 (A)
- new net: RN9.5 (R4.2), U17.13 (Qa)
- new net: RN9.6 (R3.2), U17.12 (Qb)
- new net: RN9.7 (R2.2), U17.11 (Qc)
- new net: RN9.8 (R1.2), U17.10 (Qd)
- new net: RN1.8 (R1.2), U11.10 (Qd)
- new net: RN1.7 (R2.2), U11.11 (Qc)
- new net: RN1.6 (R3.2), U11.12 (Qb)
- new net: RN1.5 (R4.2), U11.13 (Qa)
- new net: RN2.7 (R2.2), U11.14 (Qg)
- new net: RN2.6 (R3.2), U11.15 (Qf)
- new net: RN2.5 (R4.2), U11.9 (Qe)
- new net: RN27.1 (R1.1), U24.7 (DP)
- new net: RN27.2 (R2.1), U24.3 (G)
- new net: RN27.3 (R3.1), U24.2 (F)
- new net: RN27.4 (R4.1), U24.4 (E)
- new net: Q13.3 (D), U21.1 (CA), U21.6 (CA)
- new net: RN11.4 (R4.1), U21.10 (A)
- new net: RN12.3 (R3.1), U21.2 (F)
- new net: RN12.2 (R2.1), U21.3 (G)
- new net: RN12.4 (R4.1), U21.4 (E)
- new net: RN11.1 (R1.1), U21.5 (D)
- new net: RN12.1 (R1.1), U21.7 (DP)
- new net: RN11.2 (R2.1), U21.8 (C)
- new net: RN11.3 (R3.1), U21.9 (B)
- new net: RN30.4 (R4.1), U26.10 (A)
- new net: RN30.1 (R1.1), U26.5 (D)
- new net: RN30.2 (R2.1), U26.8 (C)
- new net: RN30.3 (R3.1), U26.9 (B)
- new net: Q1.3 (D), U24.1 (CA), U24.6 (CA)
- new net: RN26.4 (R4.1), U24.10 (A)
- new net: RN26.1 (R1.1), U24.5 (D)
- new net: RN26.2 (R2.1), U24.8 (C)
- new net: RN26.3 (R3.1), U24.9 (B)
- new net: RN3.1 (R1.1), U14.5 (D)
- new net: RN3.2 (R2.1), U14.8 (C)
- new net: RN3.3 (R3.1), U14.9 (B)
- new net: RN3.4 (R4.1), U14.10 (A)
- new net: RN3.5 (R4.2), U12.13 (Qa)
- new net: RN3.6 (R3.2), U12.12 (Qb)
- new net: RN3.7 (R2.2), U12.11 (Qc)
- new net: RN3.8 (R1.2), U12.10 (Qd)
- new net: Q4.1 (G), R9.2
- new net: Q4.3 (D), U25.1 (CA), U25.6 (CA)
- new net: Q1.1 (G), R6.2
- new net: RN8.7 (R2.2), U16.14 (Qg)
- new net: RN8.6 (R3.2), U16.15 (Qf)
- new net: RN8.5 (R4.2), U16.9 (Qe)
- new net: Q2.1 (G), R7.2
- new net: Q11.1 (G), R11.2
- new net: Q11.3 (D), U14.1 (CA), U14.6 (CA)
- new net: RN6.1 (R1.1), U15.7 (DP)
- new net: RN6.2 (R2.1), U15.3 (G)
- new net: RN6.3 (R3.1), U15.2 (F)
- new net: RN6.4 (R4.1), U15.4 (E)
- new net: RN6.5 (R4.2), U13.9 (Qe)
- new net: RN6.6 (R3.2), U13.15 (Qf)
- new net: RN6.7 (R2.2), U13.14 (Qg)
- new net: Q13.1 (G), R13.2
- new net: Q10.3 (D), U20.1 (CA), U20.6 (CA)
- new net: RN10.3 (R3.1), U20.2 (F)
- new net: RN10.2 (R2.1), U20.3 (G)
- new net: RN10.4 (R4.1), U20.4 (E)
- new net: RN10.1 (R1.1), U20.7 (DP)
- new net: RN28.4 (R4.1), U25.10 (A)
- new net: RN29.3 (R3.1), U25.2 (F)
- new net: RN29.2 (R2.1), U25.3 (G)
- new net: RN29.4 (R4.1), U25.4 (E)
- new net: RN28.1 (R1.1), U25.5 (D)
- new net: RN29.1 (R1.1), U25.7 (DP)
- new net: RN28.2 (R2.1), U25.8 (C)
- new net: RN28.3 (R3.1), U25.9 (B)
- new net: Q10.1 (G), R10.2
- new net: RN11.8 (R1.2), U18.10 (Qd)
- new net: RN11.7 (R2.2), U18.11 (Qc)
- new net: RN11.6 (R3.2), U18.12 (Qb)
- new net: RN11.5 (R4.2), U18.13 (Qa)
- new net: RN12.7 (R2.2), U18.14 (Qg)
- new net: RN12.6 (R3.2), U18.15 (Qf)
- new net: RN12.5 (R4.2), U18.9 (Qe)
- new net: RN8.1 (R1.1), U19.7 (DP)
- new net: RN8.2 (R2.1), U19.3 (G)
- new net: RN8.3 (R3.1), U19.2 (F)
- new net: RN8.4 (R4.1), U19.4 (E)
- new net: RN5.1 (R1.1), U15.5 (D)
- new net: RN5.2 (R2.1), U15.8 (C)
- new net: RN5.3 (R3.1), U15.9 (B)
- new net: RN5.4 (R4.1), U15.10 (A)
- new net: RN5.5 (R4.2), U13.13 (Qa)
- new net: RN5.6 (R3.2), U13.12 (Qb)
- new net: RN5.7 (R2.2), U13.11 (Qc)
- new net: RN5.8 (R1.2), U13.10 (Qd)
- new net: Q3.3 (D), U10.1 (CA), U10.6 (CA)
- new net: RN1.4 (R4.1), U10.10 (A)
- new net: RN2.3 (R3.1), U10.2 (F)
- new net: RN2.2 (R2.1), U10.3 (G)
- new net: RN2.4 (R4.1), U10.4 (E)
- new net: RN1.1 (R1.1), U10.5 (D)
- new net: RN2.1 (R1.1), U10.7 (DP)
- new net: RN1.2 (R2.1), U10.8 (C)
- new net: RN1.3 (R3.1), U10.9 (B)
- new net: Q3.1 (G), R8.2
- new net: RN4.1 (R1.1), U14.7 (DP)
- new net: RN4.2 (R2.1), U14.3 (G)
- new net: RN4.3 (R3.1), U14.2 (F)
- new net: RN4.4 (R4.1), U14.4 (E)
- new net: RN4.5 (R4.2), U12.9 (Qe)
- new net: RN4.6 (R3.2), U12.15 (Qf)
- new net: RN4.7 (R2.2), U12.14 (Qg)
- new net: RN10.7 (R2.2), U17.14 (Qg)
- new net: RN10.6 (R3.2), U17.15 (Qf)
- new net: RN10.5 (R4.2), U17.9 (Qe)
- new net: Q2.3 (D), U19.1 (CA), U19.6 (CA)
- new net OE: U40.13 (~{OE}), U41.13 (~{OE}), U42.13 (~{OE}), U43.13 (~{OE}), U44.13 (~{OE}), U45.13 (~{OE}), U46.13 (~{OE})
- new net PWM_OD: R10.1, R11.1, R13.1, R14.1, R7.1, R8.1
- new net PWM_VEL: R12.1, R6.1, R9.1
- new net RCLK: U40.12 (RCLK), U41.12 (RCLK), U42.12 (RCLK), U43.12 (RCLK), U44.12 (RCLK), U45.12 (RCLK), U46.12 (RCLK)
- new net SER: U40.14 (SER), U40.9 (QH'), U41.14 (SER), U41.9 (QH'), U42.14 (SER), U42.9 (QH'), U43.14 (SER), U43.9 (QH'), U44.14 (SER), U44.9 (QH'), U45.14 (SER), U45.9 (QH'), U46.14 (SER)
- new net SRCLK: U40.11 (SRCLK), U41.11 (SRCLK), U42.11 (SRCLK), U43.11 (SRCLK), U44.11 (SRCLK), U45.11 (SRCLK), U46.11 (SRCLK)
- new net SRCLR: U40.10 (~{SRCLR}), U41.10 (~{SRCLR}), U42.10 (~{SRCLR}), U43.10 (~{SRCLR}), U44.10 (~{SRCLR}), U45.10 (~{SRCLR}), U46.10 (~{SRCLR})
- new net S_7S_D_1_A: U18.7 (DA), U40.15 (QA)
- new net S_7S_D_1_B: U18.1 (DB), U40.1 (QB)
- new net S_7S_D_1_BI: U18.4 (~{BI}), U40.5 (QF)
- new net S_7S_D_1_C: U18.2 (DC), U40.2 (QC)
- new net S_7S_D_1_D: U18.6 (DD), U40.3 (QD)
- new net S_7S_D_1_LT: U18.3 (~{LT}), U40.4 (QE)
- new net S_7S_D_2_A: U11.7 (DA), U40.6 (QG)
- new net S_7S_D_2_B: U11.1 (DB), U40.7 (QH)
- new net S_7S_D_2_BI: U11.4 (~{BI}), U41.3 (QD)
- new net S_7S_D_2_C: U11.2 (DC), U41.15 (QA)
- new net S_7S_D_2_D: U11.6 (DD), U41.1 (QB)
- new net S_7S_D_2_LT: U11.3 (~{LT}), U41.2 (QC)
- new net S_7S_D_3_A: U16.7 (DA), U41.4 (QE)
- new net S_7S_D_3_B: U16.1 (DB), U41.5 (QF)
- new net S_7S_D_3_BI: U16.4 (~{BI}), U42.1 (QB)
- new net S_7S_D_3_C: U16.2 (DC), U41.6 (QG)
- new net S_7S_D_3_D: U16.6 (DD), U41.7 (QH)
- new net S_7S_D_3_LT: U16.3 (~{LT}), U42.15 (QA)
- new net S_7S_D_4_A: U17.7 (DA), U42.2 (QC)
- new net S_7S_D_4_B: U17.1 (DB), U42.3 (QD)
- new net S_7S_D_4_BI: U17.4 (~{BI}), U42.7 (QH)
- new net S_7S_D_4_C: U17.2 (DC), U42.4 (QE)
- new net S_7S_D_4_D: U17.6 (DD), U42.5 (QF)
- new net S_7S_D_4_LT: U17.3 (~{LT}), U42.6 (QG)
- new net S_7S_D_5_A: U12.7 (DA), U43.15 (QA)
- new net S_7S_D_5_B: U12.1 (DB), U43.1 (QB)
- new net S_7S_D_5_BI: U12.4 (~{BI}), U43.5 (QF)
- new net S_7S_D_5_C: U12.2 (DC), U43.2 (QC)
- new net S_7S_D_5_D: U12.6 (DD), U43.3 (QD)
- new net S_7S_D_5_LT: U12.3 (~{LT}), U43.4 (QE)
- new net S_7S_D_6_A: U13.7 (DA), U43.6 (QG)
- new net S_7S_D_6_B: U13.1 (DB), U43.7 (QH)
- new net S_7S_D_6_BI: U13.4 (~{BI}), U44.3 (QD)
- new net S_7S_D_6_C: U13.2 (DC), U44.15 (QA)
- new net S_7S_D_6_D: U13.6 (DD), U44.1 (QB)
- new net S_7S_D_6_LT: U13.3 (~{LT}), U44.2 (QC)
Other:
- note added: "1"
- note added: "2"
- note added: "3"
- note added: "4"
- note added: "5"
- note added: "6"
- note added: "SCH Binds"
- note added: "S_7S_A__{X}"
- note added: "S_7S_B__{X}"
- note added: "S_7S_C__{X}"
- note added: "S_7S_D_n_{X}"
- title: (none) -> Speedometer
- moved on the sheet: D58, U4, U5, U6
