File: pcb/v1/v1.kicad_pcb (KiCad board)
At the start: 2 copper layers, 60 parts, among them U4 4511, U5 4511, U6 4511

Commit message: end v1, move to modular design
Parts:
- added BAR1: HDSP-4830_2, Display:HDSP-4830, F.Cu at (220.8, 76.4)
- added BAR2: HDSP-4830_2, Display:HDSP-4830, F.Cu at (260.3, 76.2)
- added BAR3: HDSP-4830_2, Display:HDSP-4830, F.Cu at (260.8, 116.4)
- added C1: 100nF, Capacitor_SMD:C_0805_2012Metric, B.Cu at (48.5, 115.5)
- added C10: 100nF, Capacitor_SMD:C_0805_2012Metric, B.Cu at (48.5, 73.2)
- added C11: 100nF, Capacitor_SMD:C_0805_2012Metric, B.Cu at (51.2, 68.8)
- added C12: 100nF, Capacitor_SMD:C_0805_2012Metric, B.Cu at (55.0, 65.2)
- added C13: 100nF, Capacitor_SMD:C_0805_2012Metric, B.Cu at (58.5, 62.0)
- added C14: 100nF, Capacitor_SMD:C_0805_2012Metric, B.Cu at (62.8, 58.5)
- added C15: 100nF, Capacitor_SMD:C_0805_2012Metric, B.Cu at (67.5, 56.2)
- added C16: 100nF, Capacitor_SMD:C_0805_2012Metric, B.Cu at (72.0, 54.5)
- added C17: 100nF, Capacitor_SMD:C_0805_2012Metric, B.Cu at (77.0, 53.0)
- added C18: 100nF, Capacitor_SMD:C_0805_2012Metric, B.Cu at (81.5, 52.0)
- added C19: 100nF, Capacitor_SMD:C_0805_2012Metric, B.Cu at (85.8, 51.8)
- added C2: 100nF, Capacitor_SMD:C_0805_2012Metric, B.Cu at (44.8, 111.5)
- added C20: 100nF, Capacitor_SMD:C_0805_2012Metric, B.Cu at (90.0, 51.8)
- added C21: 100nF, Capacitor_SMD:C_0805_2012Metric, B.Cu at (94.8, 52.5)
- added C22: 100nF, Capacitor_SMD:C_0805_2012Metric, B.Cu at (100.0, 53.8)
- added C23: 100nF, Capacitor_SMD:C_0805_2012Metric, B.Cu at (104.5, 55.2)
- added C24: 100nF, Capacitor_SMD:C_0805_2012Metric, B.Cu at (108.5, 57.0)
- added C25: 100nF, Capacitor_SMD:C_0805_2012Metric, B.Cu at (112.2, 58.8)
- added C26: 100nF, Capacitor_SMD:C_0805_2012Metric, B.Cu at (115.5, 61.5)
- added C27: 100nF, Capacitor_SMD:C_0805_2012Metric, B.Cu at (118.4, 65.0)
- added C28: 100nF, Capacitor_SMD:C_0805_2012Metric, B.Cu at (120.8, 68.7)
- added C29: 100nF, Capacitor_SMD:C_0805_2012Metric, B.Cu at (123.2, 71.9)
- added C3: 100nF, Capacitor_SMD:C_0805_2012Metric, B.Cu at (43.0, 106.8)
- added C30: 100nF, Capacitor_SMD:C_0805_2012Metric, B.Cu at (125.3, 75.2)
- added C31: 100nF, Capacitor_SMD:C_0805_2012Metric, B.Cu at (126.7, 79.2)
- added C32: 100nF, Capacitor_SMD:C_0805_2012Metric, B.Cu at (129.3, 85.1)
- added C33: 100nF, Capacitor_SMD:C_0805_2012Metric, B.Cu at (129.8, 89.4)
- added C34: 100nF, Capacitor_SMD:C_0805_2012Metric, B.Cu at (130.6, 94.0)
- added C35: 100nF, Capacitor_SMD:C_0805_2012Metric, B.Cu at (130.3, 99.3)
- added C36: 100nF, Capacitor_SMD:C_0805_2012Metric, B.Cu at (129.5, 103.9)
- added C37: 100nF, Capacitor_SMD:C_0805_2012Metric, B.Cu at (128.3, 108.2)
- added C38: 100nF, Capacitor_SMD:C_0805_2012Metric, B.Cu at (126.5, 112.5)
- added C39: 100nF, Capacitor_SMD:C_0805_2012Metric, B.Cu at (124.7, 117.1)
- added C4: 100nF, Capacitor_SMD:C_0805_2012Metric, B.Cu at (42.2, 101.8)
- added C40: 100nF, Capacitor_SMD:C_0805_2012Metric, B.Cu at (121.7, 121.4)
- added C41: 100nF, Capacitor_SMD:C_0805_2012Metric, B.Cu at (118.1, 124.7)
- added C42: 100nF, Capacitor_SMD:C_0805_2012Metric, F.Cu at (107.0, 145.2)
- added C43: 1uF, Capacitor_SMD:C_0805_2012Metric, F.Cu at (79.9, 138.6)
- added C44: 100nF, Capacitor_SMD:C_0805_2012Metric, F.Cu at (79.9, 141.6)
- added C45: 100nF, Capacitor_SMD:C_0805_2012Metric, F.Cu at (69.5, 149.4)
- added C46: 100nF, Capacitor_SMD:C_0805_2012Metric, F.Cu at (73.9, 146.3)
- added C47: 100nF, Capacitor_SMD:C_0805_2012Metric, F.Cu at (117.8, 136.9)
- added C48: 100nF, Capacitor_SMD:C_0805_2012Metric, F.Cu at (113.4, 139.9)
- added C49: 100nF, Capacitor_SMD:C_0805_2012Metric, F.Cu at (111.4, 145.2)
- added C5: 100nF, Capacitor_SMD:C_0805_2012Metric, B.Cu at (42.2, 96.8)
- added C50: 4.7uF, Capacitor_SMD:C_0805_2012Metric, F.Cu at (69.5, 146.3)
- added C51: 100nF, Capacitor_SMD:C_0805_2012Metric, F.Cu at (122.3, 133.9)
- added C52: 2.2uF, Capacitor_SMD:C_0805_2012Metric, F.Cu at (79.9, 144.6)
- added C53: 2.2uF, Capacitor_SMD:C_0805_2012Metric, F.Cu at (74.2, 138.3)
- added C54: 100nF, Capacitor_SMD:C_0805_2012Metric, F.Cu at (74.2, 141.3)
- added C55: 15pF, Capacitor_SMD:C_0805_2012Metric, F.Cu at (91.0, 134.0)
- added C56: 15pF, Capacitor_SMD:C_0805_2012Metric, F.Cu at (107.0, 148.2)
- added C6: 100nF, Capacitor_SMD:C_0805_2012Metric, B.Cu at (42.5, 92.2)
- added C61: 47nF, Capacitor_SMD:C_0603_1608Metric, F.Cu at (84.2, 144.8)
- added C62: 0.1uF, Capacitor_SMD:C_0603_1608Metric, F.Cu at (61.3, 37.1)
- added C63: 100nF, Capacitor_SMD:C_0805_2012Metric, F.Cu at (113.4, 133.9)
- added C64: 100nF, Capacitor_SMD:C_0805_2012Metric, F.Cu at (73.9, 149.4)
- added C65: 100nF, Capacitor_SMD:C_0805_2012Metric, F.Cu at (113.4, 136.9)
- added C66: 4.7nF, Capacitor_SMD:C_0805_2012Metric, F.Cu at (84.4, 138.5)
- added C7: 100nF, Capacitor_SMD:C_0805_2012Metric, B.Cu at (43.5, 88.0)
- added C8: 100nF, Capacitor_SMD:C_0805_2012Metric, B.Cu at (44.5, 82.8)
- added C9: 100nF, Capacitor_SMD:C_0805_2012Metric, B.Cu at (46.2, 77.8)
- added D59: LED, LED_SMD:LED_0805_2012Metric_Castellated, F.Cu at (84.3, 149.3)
- added D60: LED, LED_SMD:LED_0805_2012Metric_Castellated, F.Cu at (89.2, 149.3)
- added D61: LED, LED_SMD:LED_0805_2012Metric_Castellated, F.Cu at (267.8, 153.8)
- added D62: LED, LED_SMD:LED_0805_2012Metric_Castellated, F.Cu at (259.4, 68.4)
- added D63: LED, LED_SMD:LED_0805_2012Metric_Castellated, F.Cu at (94.0, 149.3)
- added D64: LED, LED_SMD:LED_0805_2012Metric_Castellated, F.Cu at (265.2, 102.9)
- added D65: SMAJ58CA, Diode_SMD:D_SMA, F.Cu at (42.1, 49.9)
- added D66: 1N4148, Diode_SMD:D_0805_2012Metric, F.Cu at (120.4, 148.5)
- added D67: 1N4148, Diode_SMD:D_0805_2012Metric, F.Cu at (86.6, 133.2)
- added FUEL1: LTS-6980HR, Display_7Segment:7SegmentLED_LTS6760_LTS6780, F.Cu at (226.7, 136.6)
- added FUEL2: LTS-6980HR, Display_7Segment:7SegmentLED_LTS6760_LTS6780, F.Cu at (213.4, 136.6)
- added G***: LOGO, DashDash:rpm_0v7, F.Cu at (85.5, 78.2)
- added J1: USB_B, Connector_USB:USB_B_OST_USB-B1HSxx_Horizontal, F.Cu at (259.8, 42.4)
- added JP1: Jumper_NO_Small, Jumper:SolderJumper-2_P1.3mm_Open_TrianglePad1.0x1.5mm, F.Cu at (84.3, 141.7)
- added Q1: BSS138, Package_TO_SOT_SMD:SOT-23, F.Cu at (225.8, 58.0)
- added Q10: BSS138, Package_TO_SOT_SMD:SOT-23, F.Cu at (162.7, 147.3)
- added Q11: BSS138, Package_TO_SOT_SMD:SOT-23, F.Cu at (154.7, 147.3)
- added Q12: BSS138, Package_TO_SOT_SMD:SOT-23, F.Cu at (183.3, 55.1)
- added Q13: BSS138, Package_TO_SOT_SMD:SOT-23, F.Cu at (186.8, 147.3)
- added Q14: BSS138, Package_TO_SOT_SMD:SOT-23, F.Cu at (146.7, 147.3)
- added Q15: BSS138, Package_TO_SOT_SMD:SOT-23, F.Cu at (57.8, 130.3)
- added Q16: BSS138, Package_TO_SOT_SMD:SOT-23, F.Cu at (43.2, 145.0)
- added Q17: BSS138, Package_TO_SOT_SMD:SOT-23, F.Cu at (52.9, 136.2)
- added Q18: BSS138, Package_TO_SOT_SMD:SOT-23, F.Cu at (48.1, 139.1)
- added Q19: BSS138, Package_TO_SOT_SMD:SOT-23, F.Cu at (38.4, 147.9)
- added Q2: BSS138, Package_TO_SOT_SMD:SOT-23, F.Cu at (170.7, 147.3)
- added Q20: IRF540N, Package_TO_SOT_THT:TO-220-3_Vertical, F.Cu at (70.1, 26.8)
- added Q21: IRF540N, Package_TO_SOT_THT:TO-220-3_Vertical, F.Cu at (55.8, 26.9)
- added Q22: 2N3904, Package_TO_SOT_SMD:TSOT-23, F.Cu at (123.9, 143.4)
- added Q3: BSS138, Package_TO_SOT_SMD:SOT-23, F.Cu at (178.7, 147.3)
- added Q4: BSS138, Package_TO_SOT_SMD:SOT-23, F.Cu at (176.8, 29.6)
- added Q5: BSS138, Package_TO_SOT_SMD:SOT-23, F.Cu at (225.2, 150.7)
- added Q6: BSS138, Package_TO_SOT_SMD:SOT-23, F.Cu at (220.9, 142.2)
- added Q7: BSS138, Package_TO_SOT_SMD:SOT-23, F.Cu at (275.9, 138.4)
- added Q8: BSS138, Package_TO_SOT_SMD:SOT-23, F.Cu at (237.6, 96.5)
- added Q9: BSS138, Package_TO_SOT_SMD:SOT-23, F.Cu at (275.8, 99.5)
- added R1: 1k 1/10W +-1%, Resistor_SMD:R_0603_1608Metric, F.Cu at (220.1, 152.2)
- added R10: 1k 1/10W +-1%, Resistor_SMD:R_0603_1608Metric, F.Cu at (158.7, 147.5)
- added R11: 1k 1/10W +-1%, Resistor_SMD:R_0603_1608Metric, F.Cu at (150.7, 147.5)
- added R12: 1k 1/10W +-1%, Resistor_SMD:R_0603_1608Metric, F.Cu at (186.4, 50.2)
- added R13: 1k 1/10W +-1%, Resistor_SMD:R_0603_1608Metric, F.Cu at (182.6, 147.5)
- added R14: 1k 1/10W +-1%, Resistor_SMD:R_0603_1608Metric, F.Cu at (142.7, 147.6)
- added R15: 1k 1/10W +-1%, Resistor_SMD:R_0603_1608Metric, F.Cu at (42.6, 148.5)
- added R16: 1k 1/10W +-1%, Resistor_SMD:R_0603_1608Metric, F.Cu at (57.5, 133.8)
- added R17: 1k 1/10W +-1%, Resistor_SMD:R_0603_1608Metric, F.Cu at (62.0, 131.8)
- added R18: 1k 1/10W +-1%, Resistor_SMD:R_0603_1608Metric, F.Cu at (47.5, 147.7)
- added R19: 1k 1/10W +-1%, Resistor_SMD:R_0603_1608Metric, F.Cu at (52.3, 139.7)
- added R2: 1k 1/10W +-1%, Resistor_SMD:R_0603_1608Metric, F.Cu at (225.3, 141.2)
- added R20: 1k 1/10W +-1%, Resistor_SMD:R_0603_1608Metric, F.Cu at (62.0, 129.3)
- added R21: 1k 1/10W +-1%, Resistor_SMD:R_0603_1608Metric, F.Cu at (57.1, 136.3)
- added R22: 1k 1/10W +-1%, Resistor_SMD:R_0603_1608Metric, F.Cu at (47.9, 142.6)
- added R23: 1k 1/10W +-1%, Resistor_SMD:R_0603_1608Metric, F.Cu at (52.3, 142.2)
- added R24: 1k 1/10W +-1%, Resistor_SMD:R_0603_1608Metric, F.Cu at (47.5, 145.1)
- added R25: 10k, Resistor_SMD:R_0603_1608Metric, F.Cu at (176.1, 73.7)
- added R26: 0.01R, Resistor_SMD:R_1210_3225Metric, F.Cu at (111.9, 31.2)
- added R27: 57.6K 1/10W, Resistor_SMD:R_0603_1608Metric, F.Cu at (88.6, 139.3)
- added R28: 4.99K 1/10W, Resistor_SMD:R_0603_1608Metric, F.Cu at (108.9, 150.9)
- added R29: 10R 1/10W, Resistor_SMD:R_0603_1608Metric, F.Cu at (122.1, 136.7)
- added R3: 1k 1/10W +-1%, Resistor_SMD:R_0603_1608Metric, F.Cu at (277.2, 132.7)
- added R30: 10R 1/10W, Resistor_SMD:R_0603_1608Metric, F.Cu at (88.6, 136.8)
- added R31: 1M 1/10W, Resistor_SMD:R_0603_1608Metric, F.Cu at (115.6, 143.8)
- added R32: R_Small, Resistor_SMD:R_0603_1608Metric, F.Cu at (78.2, 149.8)
- added R33: R_Small, Resistor_SMD:R_0603_1608Metric, F.Cu at (82.2, 147.3)
- added R34: 10K 1/10W, Resistor_SMD:R_0603_1608Metric, F.Cu at (78.2, 147.3)
- added R35: 22R, Resistor_SMD:R_1206_3216Metric, F.Cu at (106.3, 32.9)
- added R36: 22R, Resistor_SMD:R_1206_3216Metric, F.Cu at (106.3, 29.6)
- added R4: 1k 1/10W +-1%, Resistor_SMD:R_0603_1608Metric, F.Cu at (235.9, 84.9)
- added R5: 1k 1/10W +-1%, Resistor_SMD:R_0603_1608Metric, F.Cu at (273.1, 92.1)
- added R6: 1k 1/10W +-1%, Resistor_SMD:R_0603_1608Metric, F.Cu at (233.6, 58.3)
- added R7: 1k 1/10W +-1%, Resistor_SMD:R_0603_1608Metric, F.Cu at (166.7, 147.6)
- added R8: 1k 1/10W +-1%, Resistor_SMD:R_0603_1608Metric, F.Cu at (174.7, 147.5)
- added R9: 1k 1/10W +-1%, Resistor_SMD:R_0603_1608Metric, F.Cu at (176.7, 32.2)
- added RN1: 560Ω ±5% 63mW, Resistor_SMD:R_Array_Convex_4x0603, F.Cu at (178.3, 128.5)
- added RN10: 560Ω ±5% 63mW, Resistor_SMD:R_Array_Convex_4x0603, F.Cu at (158.6, 128.5)
- added RN11: 560Ω ±5% 63mW, Resistor_SMD:R_Array_Convex_4x0603, F.Cu at (186.5, 128.5)
- added RN12: 560Ω ±5% 63mW, Resistor_SMD:R_Array_Convex_4x0603, F.Cu at (182.4, 128.5)
- added RN13: 560Ω ±5% 63mW, Resistor_SMD:R_Array_Convex_4x0603, F.Cu at (211.4, 80.2)
- added RN14: 560Ω ±5% 63mW, Resistor_SMD:R_Array_Convex_4x0603, F.Cu at (251.1, 119.2)
- added RN15: 560Ω ±5% 63mW, Resistor_SMD:R_Array_Convex_4x0603, F.Cu at (251.1, 80.5)
- added RN16: 560Ω ±5% 63mW, Resistor_SMD:R_Array_Convex_4x0603, F.Cu at (209.5, 91.0)
- added RN17: 560Ω ±5% 63mW, Resistor_SMD:R_Array_Convex_4x0603, F.Cu at (252.3, 143.2)
- added RN18: 560Ω ±5% 63mW, Resistor_SMD:R_Array_Convex_4x0603, F.Cu at (239.9, 142.0)
- added RN19: 560Ω ±5% 63mW, Resistor_SMD:R_Array_Convex_4x0603, F.Cu at (216.0, 144.5)
- added RN2: 560Ω ±5% 63mW, Resistor_SMD:R_Array_Convex_4x0603, F.Cu at (174.4, 128.5)
- added RN20: 560Ω ±5% 63mW, Resistor_SMD:R_Array_Convex_4x0603, F.Cu at (252.4, 71.7)
- added RN21: 560Ω ±5% 63mW, Resistor_SMD:R_Array_Convex_4x0603, F.Cu at (211.8, 102.6)
- added RN22: 560Ω ±5% 63mW, Resistor_SMD:R_Array_Convex_4x0603, F.Cu at (264.1, 147.6)
- added RN23: 560Ω ±5% 63mW, Resistor_SMD:R_Array_Convex_4x0603, F.Cu at (231.1, 142.9)
- added RN24: 560Ω ±5% 63mW, Resistor_SMD:R_Array_Convex_4x0603, F.Cu at (209.6, 143.4)
- added RN25: 560Ω ±5% 63mW, Resistor_SMD:R_Array_Convex_4x0603, F.Cu at (252.3, 98.0)
- added RN26: 560Ω ±5% 63mW, Resistor_SMD:R_Array_Convex_4x0603, F.Cu at (222.9, 37.1)
- added RN27: 560Ω ±5% 63mW, Resistor_SMD:R_Array_Convex_4x0603, F.Cu at (216.9, 46.6)
- added RN28: 560Ω ±5% 63mW, Resistor_SMD:R_Array_Convex_4x0603, F.Cu at (164.5, 33.1)
- added RN29: 560Ω ±5% 63mW, Resistor_SMD:R_Array_Convex_4x0603, F.Cu at (166.5, 54.6)
- added RN3: 560Ω ±5% 63mW, Resistor_SMD:R_Array_Convex_4x0603, F.Cu at (154.4, 128.5)
- added RN30: 560Ω ±5% 63mW, Resistor_SMD:R_Array_Convex_4x0603, F.Cu at (186.4, 43.0)
- added RN31: 560Ω ±5% 63mW, Resistor_SMD:R_Array_Convex_4x0603, F.Cu at (196.1, 50.2)
- added RN4: 560Ω ±5% 63mW, Resistor_SMD:R_Array_Convex_4x0603, F.Cu at (150.7, 128.5)
- added RN5: 560Ω ±5% 63mW, Resistor_SMD:R_Array_Convex_4x0603, F.Cu at (146.5, 128.5)
- added RN6: 560Ω ±5% 63mW, Resistor_SMD:R_Array_Convex_4x0603, F.Cu at (142.8, 128.5)
- added RN7: 560Ω ±5% 63mW, Resistor_SMD:R_Array_Convex_4x0603, F.Cu at (170.5, 128.5)
- added RN8: 560Ω ±5% 63mW, Resistor_SMD:R_Array_Convex_4x0603, F.Cu at (166.6, 128.5)
- added RN9: 560Ω ±5% 63mW, Resistor_SMD:R_Array_Convex_4x0603, F.Cu at (162.5, 128.5)
- added SW1: SW_Push, Button_Switch_SMD:SW_SPST_TL3342, F.Cu at (147.7, 95.1)
- added TP1: TestPoint_Small, TestPoint:TestPoint_Pad_1.0x1.0mm, F.Cu at (242.1, 152.9)
- added TP2: TestPoint_Small, TestPoint:TestPoint_Pad_1.0x1.0mm, F.Cu at (202.2, 137.5)
- added TP3: BOOT0, TestPoint:TestPoint_Pad_D2.0mm, F.Cu at (179.4, 75.5)
- added TP4: BOOT1, TestPoint:TestPoint_Pad_D2.0mm, F.Cu at (184.1, 65.3)
- added U10: HDSP-7801, Display_7Segment:HDSP-7801, F.Cu at (174.0, 133.7)
- added U11: 4511, Package_SO:TSSOP-16_4.4x5mm_P0.65mm, F.Cu at (177.4, 121.3)
- added U12: 4511, Package_SO:TSSOP-16_4.4x5mm_P0.65mm, F.Cu at (153.5, 121.3)
- added U13: 4511, Package_SO:TSSOP-16_4.4x5mm_P0.65mm, F.Cu at (145.5, 121.4)
- added U14: HDSP-7801, Display_7Segment:HDSP-7801, F.Cu at (150.0, 133.8)
- added U15: HDSP-7801, Display_7Segment:HDSP-7801, F.Cu at (142.0, 133.7)
- added U16: 4511, Package_SO:TSSOP-16_4.4x5mm_P0.65mm, F.Cu at (169.6, 121.3)
- added U17: 4511, Package_SO:TSSOP-16_4.4x5mm_P0.65mm, F.Cu at (161.6, 121.3)
- added U18: 4511, Package_SO:TSSOP-16_4.4x5mm_P0.65mm, F.Cu at (185.6, 121.3)
- added U19: HDSP-7801, Display_7Segment:HDSP-7801, F.Cu at (166.0, 133.7)
- added U20: HDSP-7801, Display_7Segment:HDSP-7801, F.Cu at (158.0, 133.8)
- added U21: HDSP-7801, Display_7Segment:HDSP-7801, F.Cu at (182.0, 133.7)
- added U22: 74HC595, Package_SO:TSSOP-16_4.4x5mm_P0.65mm, F.Cu at (196.1, 96.3)
- added U23: 74HC595, Package_SO:TSSOP-16_4.4x5mm_P0.65mm, F.Cu at (199.4, 107.8)
- added U24: HDSP-7801, DashDash:SA15-11xxx, F.Cu at (210.9, 59.1)
- added U25: HDSP-7801, DashDash:SA15-11xxx, F.Cu at (162.2, 59.1)
- added U26: HDSP-7801, DashDash:SA15-11xxx, F.Cu at (186.5, 59.1)
- added U27: 4511, Package_SO:TSSOP-16_4.4x5mm_P0.65mm, F.Cu at (232.6, 152.3)
- added U28: 4511, Package_SO:TSSOP-16_4.4x5mm_P0.65mm, F.Cu at (209.3, 153.1)
- added U32: 74HC595, Package_SO:TSSOP-16_4.4x5mm_P0.65mm, F.Cu at (252.8, 90.5)
- added U33: 74HC595, Package_SO:TSSOP-16_4.4x5mm_P0.65mm, F.Cu at (249.3, 133.9)
- added U34: 74HC595, Package_SO:TSSOP-16_4.4x5mm_P0.65mm, F.Cu at (278.6, 149.5)
- added U35: 74HC595, Package_SO:TSSOP-16_4.4x5mm_P0.65mm, F.Cu at (236.5, 108.2)
- added U38: PCA9685PW, Package_SO:TSSOP-28_4.4x9.7mm_P0.65mm, F.Cu at (192.0, 81.9)
- added U40: 74HC595, Package_SO:TSSOP-16_4.4x5mm_P0.65mm, F.Cu at (183.0, 111.4)
- added U41: 74HC595, Package_SO:TSSOP-16_4.4x5mm_P0.65mm, F.Cu at (172.8, 110.9)
- added U42: 74HC595, Package_SO:TSSOP-16_4.4x5mm_P0.65mm, B.Cu at (161.7, 118.5)
- added U43: 74HC595, Package_SO:TSSOP-16_4.4x5mm_P0.65mm, F.Cu at (153.7, 111.1)
- added U44: 74HC595, Package_SO:TSSOP-16_4.4x5mm_P0.65mm, F.Cu at (145.7, 112.9)
- added U45: 74HC595, Package_SO:TSSOP-16_4.4x5mm_P0.65mm, F.Cu at (203.7, 31.9)
- added U46: 74HC595, Package_SO:TSSOP-16_4.4x5mm_P0.65mm, F.Cu at (163.4, 47.8)
- added U47: STM32F405VGTx, Package_QFP:LQFP-100_14x14mm_P0.5mm, F.Cu at (164.6, 85.9)
- added U48: 25LCxxx, Package_SO:SOIC-8_3.9x4.9mm_P1.27mm, F.Cu at (180.2, 97.3)
- added U49: MIC2940A-5.0WT, Package_TO_SOT_THT:TO-220-3_Vertical, F.Cu at (76.9, 31.8)
- added U50: MIC2940A-3.3WU, Package_TO_SOT_SMD:TO-263-3_TabPin2, F.Cu at (35.6, 37.7)
- added U51: LT4363IMS, Package_SO:SOIC-16W_7.5x10.3mm_P1.27mm, F.Cu at (51.5, 36.0)
- added U52: ADUM4160, Package_SO:SOIC-16W_7.5x10.3mm_P1.27mm, F.Cu at (266.2, 53.2)
- added U53: TJA1042T3118, Package_SO:HTSOP-8-1EP_3.9x4.9mm_P1.27mm_EP2.4x3.2mm, F.Cu at (198.8, 67.8)
- added Y1: 25MHz, Crystal:Crystal_SMD_3225-4Pin_3.2x2.5mm, F.Cu at (146.7, 79.2)
- D1, D10, D11, D12, D13, D14, D15, D16, D17, D18, D19, D2, D20, D21, D22, D23, D24, D25, D26, D27, D28, D29, D3, D30, D31, D32, D33, D34, D35, D36, D37, D38, D39, D4, D40, D41, D5, D6, D7, D8, D9: value LED -> WS2812B; footprint LED_SMD:LED_0805_2012Metric_Castellated -> LED_SMD:LED_SK6812MINI_PLCC4_3.5x3.5mm_P1.75mm
- U4, U5, U6: footprint Package_SO:SOP-16_4.55x10.3mm_P1.27mm -> Package_SO:TSSOP-16_4.4x5mm_P0.65mm
- moved U4 183.6 mm to (229.4, 50.5)
- moved U6 144.5 mm to (194.6, 38.4)
- moved U5 106.1 mm to (162.4, 39.4), turned to 90 degrees
- moved D38 88.8 mm to (126.6, 112.7), turned to -20 degrees
- moved D35 88.7 mm to (130.3, 99.2)
- moved D48 87.3 mm to (43.4, 141.2)
- moved D57 87.3 mm to (38.6, 141.2)
- moved D50 86.4 mm to (38.6, 132.4)
- moved D43 82.8 mm to (38.6, 144.2)
- moved D51 79.3 mm to (48.3, 129.5)
- moved D39 79.1 mm to (124.7, 117.1), turned to -20 degrees
- moved D34 77.3 mm to (130.5, 94.1)
- moved D52 75.3 mm to (43.4, 135.4)
- moved D56 75.3 mm to (43.4, 132.4)
- moved D36 74.4 mm to (129.7, 103.9), turned to -10 degrees
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Connections:
- D1 pad 1: /Tachometer/D1 -> +5VA
- D1 pad 2: unconnected-(D1-Pad2) -> Net-(D1-Pad2)
- D10 pad 1: /Tachometer/D10 -> +5VA
- D11 pad 1: /Tachometer/D11 -> +5VA
- D11 pad 2: Net-(D10-Pad2) -> Net-(D11-Pad2)
- D12 pad 1: /Tachometer/D12 -> +5VA
- D13 pad 1: /Tachometer/D13 -> +5VA
- D13 pad 2: Net-(D12-Pad2) -> Net-(D13-Pad2)
- D14 pad 1: /Tachometer/D14 -> +5VA
- D14 pad 2: Net-(D12-Pad2) -> Net-(D14-Pad2)
- D15 pad 1: /Tachometer/D15 -> +5VA
- D15 pad 2: Net-(D12-Pad2) -> Net-(D15-Pad2)
- D16 pad 1: /Tachometer/D16 -> +5VA
- D16 pad 2: Net-(D12-Pad2) -> Net-(D16-Pad2)
- D17 pad 1: /Tachometer/D17 -> +5VA
- D18 pad 1: /Tachometer/D18 -> +5VA
- D18 pad 2: Net-(D17-Pad2) -> Net-(D18-Pad2)
- D19 pad 1: /Tachometer/D19 -> +5VA
- D19 pad 2: Net-(D17-Pad2) -> Net-(D19-Pad2)
- D2 pad 1: /Tachometer/D2 -> +5VA
- D20 pad 1: /Tachometer/D20 -> +5VA
- D20 pad 2: Net-(D17-Pad2) -> Net-(D20-Pad2)
- D21 pad 1: /Tachometer/D21 -> +5VA
- D21 pad 2: Net-(D17-Pad2) -> Net-(D21-Pad2)
- D22 pad 1: /Tachometer/D22 -> +5VA
- D23 pad 1: /Tachometer/D23 -> +5VA
- D23 pad 2: Net-(D22-Pad2) -> Net-(D23-Pad2)
- D24 pad 1: /Tachometer/D24 -> +5VA
- D24 pad 2: Net-(D22-Pad2) -> Net-(D24-Pad2)
- D25 pad 1: /Tachometer/D25 -> +5VA
- D25 pad 2: Net-(D22-Pad2) -> Net-(D25-Pad2)
- D26 pad 1: /Tachometer/D26 -> +5VA
- D26 pad 2: Net-(D22-Pad2) -> Net-(D26-Pad2)
- D27 pad 1: /Tachometer/D27 -> Net-(C27-Pad2)
- D28 pad 1: /Tachometer/D28 -> Net-(C27-Pad2)
- D28 pad 2: Net-(D27-Pad2) -> Net-(D28-Pad2)
- D29 pad 1: /Tachometer/D29 -> Net-(C27-Pad2)
- D29 pad 2: Net-(D27-Pad2) -> Net-(D29-Pad2)
- D3 pad 1: /Tachometer/D3 -> +5VA
- D3 pad 2: Net-(D2-Pad2) -> Net-(D3-Pad2)
- D30 pad 1: /Tachometer/D30 -> Net-(C27-Pad2)
- D30 pad 2: Net-(D27-Pad2) -> Net-(D30-Pad2)
- D31 pad 1: /Tachometer/D31 -> Net-(C27-Pad2)
- D31 pad 2: Net-(D27-Pad2) -> Net-(D31-Pad2)
- D32 pad 1: /Tachometer/D32 -> +5VA
- D33 pad 1: /Tachometer/D33 -> +5VA
- D33 pad 2: Net-(D32-Pad2) -> Net-(D33-Pad2)
- D34 pad 1: /Tachometer/D34 -> +5VA
- D34 pad 2: Net-(D32-Pad2) -> Net-(D34-Pad2)
- D35 pad 1: /Tachometer/D35 -> +5VA
- D35 pad 2: Net-(D32-Pad2) -> Net-(D35-Pad2)
- D36 pad 1: /Tachometer/D36 -> +5VA
- D36 pad 2: Net-(D32-Pad2) -> Net-(D36-Pad2)
- D37 pad 1: /Tachometer/D37 -> +5VA
- D38 pad 1: /Tachometer/D38 -> +5VA
- D38 pad 2: Net-(D37-Pad2) -> Net-(D38-Pad2)
- D39 pad 1: /Tachometer/D39 -> +5VA
- D39 pad 2: Net-(D37-Pad2) -> Net-(D39-Pad2)
- D4 pad 1: /Tachometer/D4 -> +5VA
- D4 pad 2: Net-(D2-Pad2) -> Net-(D4-Pad2)
- D40 pad 1: /Tachometer/D40 -> +5VA
- D40 pad 2: Net-(D37-Pad2) -> Net-(D40-Pad2)
- D41 pad 1: /Tachometer/D41 -> +5VA
- D41 pad 2: Net-(D37-Pad2) -> unconnected-(D41-Pad2)
- D42 pad 2: Net-(D42-Pad2) -> +12V
- D43 pad 2: Net-(D42-Pad2) -> +12V
- D44 pad 2: Net-(D44-Pad2) -> Net-(D42-Pad1)
- D45 pad 2: unconnected-(D45-Pad2) -> Net-(D43-Pad1)
- D46 pad 2: unconnected-(D46-Pad2) -> Net-(D44-Pad1)
- D47 pad 2: unconnected-(D47-Pad2) -> Net-(D45-Pad1)
- D48 pad 1: /Tachometer/REV -> /TachometerV2/BA_1
- D48 pad 2: Net-(D42-Pad1) -> Net-(D46-Pad1)
- D49 pad 1: /Tachometer/LAUNCH -> /TachometerV2/BA_2
- D49 pad 2: Net-(D43-Pad1) -> Net-(D47-Pad1)
- D5 pad 1: /Tachometer/D5 -> +5VA
- D5 pad 2: Net-(D2-Pad2) -> Net-(D5-Pad2)
- D50 pad 1: /Tachometer/SHIFT -> Net-(D50-Pad1)
- D50 pad 2: Net-(D44-Pad1) -> Net-(D50-Pad2)
- D51 pad 1: Net-(D44-Pad2) -> Net-(D51-Pad1)
- D51 pad 2: Net-(D45-Pad1) -> Net-(D50-Pad2)
- D52 pad 2: Net-(D46-Pad1) -> Net-(D52-Pad2)
- D53 pad 2: Net-(D47-Pad1) -> unconnected-(D53-Pad2)
- D54 pad 1: Net-(D54-Pad1) -> /TCH_REV
- D54 pad 2: Net-(D52-Pad1) -> Net-(D50-Pad1)
- D55 pad 1: Net-(D55-Pad1) -> /TCH_LAUNCH
- D55 pad 2: Net-(D53-Pad1) -> Net-(D51-Pad1)
- D56 pad 1: /Tachometer/BA_1 -> /TCH_SHIFT
- D56 pad 2: Net-(D54-Pad1) -> Net-(D52-Pad1)
- D57 pad 1: /Tachometer/BA_2 -> Net-(D52-Pad2)
- D57 pad 2: Net-(D55-Pad1) -> Net-(D53-Pad1)
- D6 pad 1: /Tachometer/D6 -> +5VA
- D6 pad 2: Net-(D2-Pad2) -> Net-(D6-Pad2)
- D7 pad 1: /Tachometer/D7 -> +5VA
- D7 pad 2: Net-(D10-Pad2) -> Net-(D7-Pad2)
- D8 pad 1: /Tachometer/D8 -> +5VA
- D8 pad 2: Net-(D10-Pad2) -> Net-(D8-Pad2)
- D9 pad 1: /Tachometer/D9 -> +5VA
- D9 pad 2: Net-(D10-Pad2) -> Net-(D10-Pad4)
- U4 pad 1: unconnected-(U4-Pad1) -> /Speedometer/S_7S_A_DB
- U4 pad 10: unconnected-(U4-Pad10) -> Net-(RN26-Pad8)
- U4 pad 11: unconnected-(U4-Pad11) -> Net-(RN26-Pad7)
- U4 pad 12: unconnected-(U4-Pad12) -> Net-(RN26-Pad6)
- U4 pad 13: unconnected-(U4-Pad13) -> Net-(RN26-Pad5)
- U4 pad 14: unconnected-(U4-Pad14) -> Net-(RN27-Pad7)
- U4 pad 15: unconnected-(U4-Pad15) -> Net-(RN27-Pad6)
- U4 pad 16: Vdd -> +12V
- U4 pad 2: unconnected-(U4-Pad2) -> /Speedometer/S_7S_A_DC
- U4 pad 3: unconnected-(U4-Pad3) -> /Speedometer/S_7S_A_LT
- U4 pad 4: unconnected-(U4-Pad4) -> /Speedometer/S_7S_A_BI
- U4 pad 5: unconnected-(U4-Pad5) -> GND
- U4 pad 6: unconnected-(U4-Pad6) -> /Speedometer/S_7S_A_DD
- U4 pad 7: unconnected-(U4-Pad7) -> /Speedometer/S_7S_A_DA
- U4 pad 8: Vss -> GND
- U4 pad 9: unconnected-(U4-Pad9) -> Net-(RN27-Pad5)
- U5 pad 1: unconnected-(U5-Pad1) -> /Speedometer/S_7S_B_DB
- U5 pad 10: unconnected-(U5-Pad10) -> Net-(RN28-Pad8)
- U5 pad 11: unconnected-(U5-Pad11) -> Net-(RN28-Pad7)
- U5 pad 12: unconnected-(U5-Pad12) -> Net-(RN28-Pad6)
- U5 pad 13: unconnected-(U5-Pad13) -> Net-(RN28-Pad5)
- U5 pad 14: unconnected-(U5-Pad14) -> Net-(RN29-Pad7)
- U5 pad 15: unconnected-(U5-Pad15) -> Net-(RN29-Pad6)
- U5 pad 16: Vdd -> +12V
- U5 pad 2: unconnected-(U5-Pad2) -> /Speedometer/S_7S_B_DC
- U5 pad 3: unconnected-(U5-Pad3) -> /Speedometer/S_7S_B_LT
- U5 pad 4: unconnected-(U5-Pad4) -> /Speedometer/S_7S_B_BI
- U5 pad 5: unconnected-(U5-Pad5) -> GND
- U5 pad 6: unconnected-(U5-Pad6) -> /Speedometer/S_7S_B_DD
- U5 pad 7: unconnected-(U5-Pad7) -> /Speedometer/S_7S_B_DA
- U5 pad 8: Vss -> GND
- U5 pad 9: unconnected-(U5-Pad9) -> Net-(RN29-Pad5)
- U6 pad 1: unconnected-(U6-Pad1) -> /Speedometer/S_7S_B_DB
- U6 pad 10: unconnected-(U6-Pad10) -> Net-(RN30-Pad8)
- U6 pad 11: unconnected-(U6-Pad11) -> Net-(RN30-Pad7)
- U6 pad 12: unconnected-(U6-Pad12) -> Net-(RN30-Pad6)
- U6 pad 13: unconnected-(U6-Pad13) -> Net-(RN30-Pad5)
- U6 pad 14: unconnected-(U6-Pad14) -> Net-(RN31-Pad7)
- U6 pad 15: unconnected-(U6-Pad15) -> Net-(RN31-Pad6)
- U6 pad 16: Vdd -> +12V
- U6 pad 2: unconnected-(U6-Pad2) -> /Speedometer/S_7S_B_DC
- U6 pad 3: unconnected-(U6-Pad3) -> /Speedometer/S_7S_B_LT
- U6 pad 4: unconnected-(U6-Pad4) -> /Speedometer/S_7S_B_BI
- U6 pad 5: unconnected-(U6-Pad5) -> GND
- U6 pad 6: unconnected-(U6-Pad6) -> /Speedometer/S_7S_B_DD
- U6 pad 7: unconnected-(U6-Pad7) -> /Speedometer/S_7S_B_DA
- U6 pad 8: Vss -> GND
- U6 pad 9: unconnected-(U6-Pad9) -> Net-(RN31-Pad5)
Routing:
- net /PWM_OD: track 0.00 -> 47.1 mm
- net Net-(RN5-Pad1): track 0.00 -> 16.6 mm
- net Net-(RN8-Pad1): track 0.00 -> 16.4 mm, vias 0 -> 1
- net Net-(RN12-Pad1): track 0.00 -> 16.3 mm, vias 0 -> 1
- net Net-(RN2-Pad1): track 0.00 -> 16.1 mm, vias 0 -> 1
- net Net-(RN6-Pad1): track 0.00 -> 16.1 mm, vias 0 -> 1
- net Net-(RN9-Pad1): track 0.00 -> 15.9 mm
- net Net-(RN7-Pad1): track 0.00 -> 15.9 mm
- net Net-(RN11-Pad1): track 0.00 -> 15.9 mm
- net Net-(RN3-Pad1): track 0.00 -> 15.9 mm
- net Net-(RN10-Pad1): track 0.00 -> 15.8 mm, vias 0 -> 1
- net Net-(RN1-Pad1): track 0.00 -> 15.8 mm
- net Net-(RN4-Pad1): track 0.00 -> 15.4 mm, vias 0 -> 1
- net Net-(Q14-Pad3): track 0.00 -> 14.8 mm
- net Net-(Q2-Pad3): track 0.00 -> 14.8 mm
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Other:
- board outline added: 265.5 x 132.2 mm
- board text added: "Battery"
- board text added: "Fuel"
- board text added: "Oil Pres"
- board text added: "TBD: Conector I/O"
- board text added: "Temp"
