File: pcb/v1/v1.kicad_sch (KiCad schematic)
At the start: 0 parts

Commit message: end v1, move to modular design
Parts:
- added C42, C44, C45, C46, C47, C48, C49, C51, C54, C63, C64, C65: 100nF, Capacitor_SMD:C_0805_2012Metric, symbol Device:C_Small
- added C43: 1uF, Capacitor_SMD:C_0805_2012Metric, symbol Device:C_Small
- added C50: 4.7uF, Capacitor_SMD:C_0805_2012Metric, symbol Device:CP_Small
- added C52, C53: 2.2uF, Capacitor_SMD:C_0805_2012Metric, symbol Device:C_Small
- added C55, C56: 15pF, Capacitor_SMD:C_0805_2012Metric, symbol Device:C_Small
- added C57, C58, C59, C60: CP_Small, symbol Device:CP_Small
- added C61: 47nF, Capacitor_SMD:C_0603_1608Metric, symbol Device:C_Small
- added C62: 0.1uF, Capacitor_SMD:C_0603_1608Metric, symbol Device:C_Small
- added C66: 4.7nF, Capacitor_SMD:C_0805_2012Metric, symbol Device:C_Small
- added D65: SMAJ58CA, Diode_SMD:D_SMA, symbol Device:D_TVS
- added D66, D67: 1N4148, Diode_SMD:D_0805_2012Metric, symbol Diode:1N4148
- added J1: USB_B, Connector_USB:USB_B_OST_USB-B1HSxx_Horizontal, symbol STM32F_rev3-rescue:USB_B-Connector
- added JP1: Jumper_NO_Small, Jumper:SolderJumper-2_P1.3mm_Open_TrianglePad1.0x1.5mm, symbol Device:Jumper_NO_Small
- added Q20, Q21: IRF540N, Package_TO_SOT_THT:TO-220-3_Vertical, symbol Transistor_FET:IRF540N
- added Q22: 2N3904, Package_TO_SOT_SMD:TSOT-23, symbol Transistor_BJT:2N3904
- added R25: 10k, Resistor_SMD:R_0603_1608Metric, symbol Device:R_Small
- added R26: 0.01R, Resistor_SMD:R_1210_3225Metric, symbol Device:R_Small
- added R27: 57.6K 1/10W, Resistor_SMD:R_0603_1608Metric, symbol Device:R_Small
- added R28: 4.99K 1/10W, Resistor_SMD:R_0603_1608Metric, symbol Device:R_Small
- added R29, R30: 10R 1/10W, Resistor_SMD:R_0603_1608Metric, symbol Device:R_Small
- added R31: 1M 1/10W, Resistor_SMD:R_0603_1608Metric, symbol Device:R_Small
- added R32, R33: R_Small, Resistor_SMD:R_0603_1608Metric, symbol Device:R_Small
- added R34: 10K 1/10W, Resistor_SMD:R_0603_1608Metric, symbol Device:R_Small
- added R35, R36: 22R, Resistor_SMD:R_1206_3216Metric, symbol Device:R_Small
- added SW1: SW_Push, Button_Switch_SMD:SW_SPST_TL3342, symbol Switch:SW_Push
- added TP3: BOOT0, TestPoint:TestPoint_Pad_D2.0mm, symbol Connector:TestPoint_Small
- added TP4: BOOT1, TestPoint:TestPoint_Pad_D2.0mm, symbol Connector:TestPoint_Small
- added U36, U37, U39: 74LS125, symbol 74xx:74LS125
- added U38: PCA9685PW, Package_SO:TSSOP-28_4.4x9.7mm_P0.65mm, symbol Driver_LED:PCA9685PW
- added U47: STM32F405VGTx, Package_QFP:LQFP-100_14x14mm_P0.5mm, symbol MCU_ST_STM32F4:STM32F405VGTx
- added U48: 25LCxxx, Package_SO:SOIC-8_3.9x4.9mm_P1.27mm, symbol Memory_EEPROM:25LCxxx
- added U49: MIC2940A-5.0WT, Package_TO_SOT_THT:TO-220-3_Vertical, symbol Regulator_Linear:L7805
- added U50: MIC2940A-3.3WU, Package_TO_SOT_SMD:TO-263-3_TabPin2, symbol Regulator_Linear:L7805
- added U51: LT4363IMS, Package_SO:SOIC-16W_7.5x10.3mm_P1.27mm, symbol OpenEFI-STM32-rev3:LT4363IMS
- added U52: ADUM4160, Package_SO:SOIC-16W_7.5x10.3mm_P1.27mm, symbol Interface_USB:ADUM4160
- added U53: TJA1042T3118, Package_SO:HTSOP-8-1EP_3.9x4.9mm_P1.27mm_EP2.4x3.2mm, symbol OpenEFI-STM32-rev3:TJA1042T3118
- added U? (x6): SensorsV2, OpenEFI-STM32F_rev3:Sensors_v2, symbol OpenEFI-STM32-rev3:SensorsV2
- added Y1: 25MHz, Crystal:Crystal_SMD_3225-4Pin_3.2x2.5mm, symbol Device:Crystal_GND24
Connections:
- new net: Q20.1 (G), R29.1
- new net: Q22.3 (C), R29.2, R31.2
- new net: Q21.1 (G), R30.1
- new net: C61.1, R30.2, R31.1, U51.4 (GATE)
- new net: D66.1 (K), Q22.2 (B), R34.1
- new net: D67.1 (K), R34.2
- new net: C63.1, J1.1 (VBUS), U52.1 (VBUS1)
- new net: C64.1, U52.3 (VDD1), U52.4 (PDEN), U52.5 (SPU)
- new net: R27.2, R28.2, U51.1 (FB)
- new net: C62.1, U51.12 (TMR)
- new net: Q21.2 (D), R26.2, U51.3 (SNS)
- new net: D65.1 (A1), Q20.2 (D), Q21.3 (S), U51.5 (VCC)
- new net: C66.1, R35.1, R36.1
- new net: TP4.1, U47.37 (PB2)
- new net: C52.1, U47.49 (VCAP_1)
- new net: C53.1, U47.73 (VCAP_2)
- new net: R25.1, TP3.1, U47.94 (BOOT0)
- new net +12V: C57.1, C59.1, JP1.2, R26.1, R27.1, U49.1 (IN), U50.1 (IN), U51.2 (OUT)
- new net +12VA: D66.2 (A), JP1.1, Q20.3 (S), Q22.1 (E)
- new net +3V3: C42.1, C43.1, C44.1, C45.1, C46.1, C47.1, C48.1, C49.1, C50.1, C54.1, C60.1, C65.1, U38.28 (VDD), U47.100 (VDD), U47.11 (VDD), U47.19 (VDD), U47.21 (VREF+), U47.22 (VDDA), U47.28 (VDD), U47.50 (VDD), U47.6 (VBAT), U47.75 (VDD), U48.3 (~{WP}), U48.7 (~{HOLD}), U48.8 (VCC), U50.3 (OUT), U52.12 (PIN), U52.13 (SPD), U52.14 (VDD2), U52.16 (VBUS2), U53.5 (VIO)
- new net +5V: C58.1, U36.14 (VCC), U37.14 (VCC), U49.3 (OUT), U53.3 (VCC)
- new net BFT_OE: U39.2, U47.38 (PE7)
- new net BFT_OE_L: U39.3
- new net BFT_RCLK: U36.9, U47.40 (PE9)
- new net BFT_RCLK_L: U36.8
- new net BFT_SER: U36.12, U47.39 (PE8)
- new net BFT_SER_L: U36.11
- new net BFT_SRCLK: U36.2, U47.42 (PE11)
- new net BFT_SRCLK_L: U36.3
- new net BFT_SRCLR: U36.5, U47.41 (PE10)
- new net BFT_SRCLR_L: U36.6
- new net CAN+: R35.2, U53.7 (CANH)
- new net CAN-: R36.2, U53.6 (CANL)
- new net CAN1_RX: U47.81 (PD0), U53.4 (RXD)
- new net CAN1_TX: U47.82 (PD1), U53.1 (TXD)
- new net D+: R32.1, U52.7 (UD+)
- new net D-: R33.1, U52.6 (UD-)
- new net GND: C42.2, C43.2, C44.2, C45.2, C46.2, C47.2, C48.2, C49.2, C50.2, C51.1, C52.2, C53.2, C54.2, C55.2, C56.2, C57.2, C58.2, C59.2, C60.2, C61.2, C62.2, C65.2, C66.2, D65.2 (A2), D67.2 (A), R25.2, R28.1, SW1.2, U36.1, U36.10, U36.13, U36.4, U36.7 (GND), U37.1, U37.10, U37.13, U37.4, U37.7 (GND), U38.1 (A0), U38.14 (VSS), U38.2 (A1), U38.23 (~{OE}), U38.24 (A5), U38.3 (A2), U38.4 (A3), U38.5 (A4), U39.1, U39.10, U39.13, U39.4, U47.10 (VSS), U47.20 (VSSA), U47.27 (VSS), U47.74 (VSS), U47.99 (VSS), U48.4 (GND), U49.2 (GND), U50.2 (GND), U51.9 (GND), U52.15 (GND2), U52.9 (GND2), U53.2 (GND), U53.8 (STB), Y1.2, Y1.4
- new net GND1: C63.2, C64.2, J1.4 (GND), J1.5 (Shield), U52.2 (GND1), U52.8 (GND1)
- new net I2C1_SCL: U38.27 (SDA), U47.92 (PB6)
- new net I2C1_SDA: U38.26 (SCL), U47.93 (PB7)
- new net MEMORY_CS: U48.1 (~{CS})
- new net NRST: C51.2, SW1.1, U47.14 (NRST)
- new net OSC_IN: C55.1, U47.12 (PH0), Y1.1
- new net OSC_OUT: C56.1, U47.13 (PH1), Y1.3
- new net PWM_BACK_1: U38.13 (LED7)
- new net PWM_BACK_2: U38.15 (LED8)
- new net PWM_BAR1: U38.8 (LED2)
- new net PWM_BAR2: U38.9 (LED3)
- new net PWM_BAR3: U38.10 (LED4)
- new net PWM_FUEL1: U38.6 (LED0)
- new net PWM_FUEL2: U38.7 (LED1)
- new net PWM_OD: U38.12 (LED6)
- new net PWM_VEL: U38.11 (LED5)
- new net SPEED_OE: U37.5, U47.58 (PD11)
- new net SPEED_OE_L: U37.6
- new net SPEED_RCLK: U39.12, U47.60 (PD13)
- new net SPEED_RCLK_L: U39.11
- new net SPEED_SER: U37.2, U47.59 (PD12)
- new net SPEED_SER_L: U37.3
- new net SPEED_SRCLK: U39.6, U47.62 (PD15)
- new net SPEED_SRCLK_L: U39.5
- new net SPEED_SRCLR: U39.9, U47.61 (PD14)
- new net SPEED_SRCLR_L: U39.8
- new net SPI2_MISO: U47.53 (PB14), U48.2 (MISO)
- new net SPI2_MOSI: U47.54 (PB15), U48.5 (MOSI)
- new net SPI2_SCK: U47.47 (PB10), U48.6 (SCK)
- new net SYS_SWCLK: U47.76 (PA14)
- new net SYS_SWDIO: U47.72 (PA13)
- new net SYS_SWO: U47.89 (PB3)
- new net TCH_DIN: U47.78 (PC10)
- new net TCH_LAUNCH: U47.65 (PC8)
- new net TCH_REV: U47.66 (PC9)
- new net TCH_SHIFT: U47.64 (PC7)
- new net USB_D+: U47.71 (PA12), U52.10 (DD+)
- new net USB_D-: U47.70 (PA11), U52.11 (DD-)
- new net VBUS: U47.68 (PA9)
- new net d+: J1.3 (D+), R32.2
- new net d-: J1.2 (D-), R33.2
- no-connect marks 0 -> 7
Other:
- removed sheet Tachometer
- added sheet Battery/Fuel/Temperature indicators (Battery-Fuel-Temperature.kicad_sch)
- added sheet TachometerV2 (TachometerV2.kicad_sch)
- sheet Speedometer ports: added OE, PWM_OD, PWM_VEL, RCLK, SER, SRCLK, SRCLR; removed none
- note added: "CAN"
- note added: "Crystal"
- note added: "DEBUG PIN"
- note added: "El Clock hace falta si me quedo sin inputs para sincronizar el segundo"
- note added: "Surge Protection (optional)"
- note added: "UNLIMITED POWAAAAA"
- note added: "USB Protection (Optional)"
- note added: "VDD Decoupling"
- note added: "VREF Decoupling"
