File: pcb/v2/dashdashv2/_autosave-dashdashv2.kicad_pcb (KiCad board)
At the start: 2 copper layers, 69 parts, among them J1 USB_B, J2 Tag connect, J3 Conn_01x04_Female, Q1 IRF540N, Q2 IRF540N, Q3 2N3904, U1 RP2040, U10 PCA9685PW, U11 MIC2940A-3.3WU, U13 LT4363IMS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

Commit message: main board sch
Parts:
- added J4: Conn_01x04_Female, Connector_Molex:Molex_Mini-Fit_Jr_5569-04A1_2x02_P4.20mm_Horizontal, F.Cu at (196.3, 83.6)
- added U5: TPD2E2U06, Package_TO_SOT_SMD:SOT-143, F.Cu at (197.0, 127.1)
- R10, R11: value R_Small -> 22r
Connections:
- J3 pad 1: unconnected-(J3-Pad1) -> GND
- J3 pad 3: unconnected-(J3-Pad3) -> CAN-
- J3 pad 4: unconnected-(J3-Pad4) -> CAN+
- R1 pad 2: /USB_DM -> /USB_D-
- R2 pad 1: /USB_DP -> /USB_D+
