File: pcb/v2/dashdashv2/dashdashv2.kicad_sch (KiCad schematic)
At the start: 65 parts, among them J1 USB_B, Q1 IRF540N, Q2 IRF540N, Q3 2N3904, SW1 SW_Push, U1 SensorsV2, U10 PCA9685PW, U11 MIC2940A-3.3WU, U12 TJA1042T3118, U13 LT4363IMS, U14 ADUM4160, U15 74LS125, U16 74LS125, U2 SensorsV2, U3 SensorsV2, U4 SensorsV2, U5 SensorsV2, U6 SensorsV2, U7 25LCxxx, U8 STM32F405VGTx, U9 MIC2940A-5.0WT, Y1 25MHz

Commit message: main board sch
Parts:
- removed C23, C24: 100nF, Capacitor_SMD:C_0805_2012Metric, symbol Device:C_Small
- removed C9: 4.7uF, Capacitor_SMD:C_0805_2012Metric, symbol Device:CP_Small
- removed R1: 10k, Resistor_SMD:R_0603_1608Metric, symbol Device:R_Small
- removed R10, R11: R_Small, Resistor_SMD:R_0603_1608Metric, symbol Device:R_Small
- removed R2, R3: 22R, Resistor_SMD:R_1206_3216Metric, symbol Device:R_Small
- removed SW1: SW_Push, Button_Switch_SMD:SW_SPST_TL3342, symbol Switch:SW_Push
- removed TP1: BOOT0, TestPoint:TestPoint_Pad_D2.0mm, symbol Connector:TestPoint_Small
- removed TP2: BOOT1, TestPoint:TestPoint_Pad_D2.0mm, symbol Connector:TestPoint_Small
- removed U1, U2, U3, U4, U5, U6: SensorsV2, OpenEFI-STM32F_rev3:SensorsV2, symbol OpenEFI-STM32-rev3:SensorsV2
- removed U12: TJA1042T3118, Package_SO:HTSOP-8-1EP_3.9x4.9mm_P1.27mm_EP2.4x3.2mm, symbol OpenEFI-STM32-rev3:TJA1042T3118
- removed U14: ADUM4160, Package_SO:SOIC-16W_7.5x10.3mm_P1.27mm, symbol Interface_USB:ADUM4160
- removed U15, U16: 74LS125, symbol 74xx:74LS125
- removed U8: STM32F405VGTx, Package_QFP:LQFP-100_14x14mm_P0.5mm, symbol MCU_ST_STM32F4:STM32F405VGTx
- added BATT_CONN1, DISPLAY1, FUEL_CONN1, O2_CONN1, OIL_CONN1, OIL_TEMP1, RPM_CONN1, SPEED_CONN1, TEMP1: Conn_01x08, symbol Connector_Generic:Conn_01x08
- added C26, C27, C28: 100nF, Capacitor_SMD:C_0603_1608Metric, symbol Device:C_Small
- added C9: 4.7nF, Capacitor_SMD:C_0805_2012Metric, symbol Device:C_Small
- added D4: GREEN, LED_SMD:LED_0603_1608Metric, symbol Device:LED
- added D5: BLUE, LED_SMD:LED_0603_1608Metric, symbol Device:LED
- added D6: RED, LED_SMD:LED_0603_1608Metric, symbol Device:LED
- added J2: Tag connect, Connector:Tag-Connect_TC2030-IDC-NL_2x03_P1.27mm_Vertical, symbol Connector_Generic:Conn_02x03_Odd_Even
- added J3, J4: Conn_01x04_Female, Connector_Molex:Molex_Mini-Fit_Jr_5569-04A1_2x02_P4.20mm_Horizontal, symbol Connector:Conn_01x04_Female
- added JP2: BOOTSEL, Jumper:SolderJumper-2_P1.3mm_Open_TrianglePad1.0x1.5mm, symbol Jumper:SolderJumper_2_Open
- added R1, R2: 27R, Resistor_SMD:R_0603_1608Metric, symbol Device:R
- added R13, R14: 10k, Resistor_SMD:R_0603_1608Metric, symbol Device:R
- added R15, R16: 30R, Resistor_SMD:R_1206_3216Metric, symbol Device:R_Small
- added R17, R18, R19, R3: 1k, Resistor_SMD:R_0603_1608Metric, symbol Device:R
- added U1: RP2040, Package_DFN_QFN:QFN-56-1EP_7x7mm_P0.4mm_EP3.2x3.2mm, symbol rp2040:RP2040
- added U2: W25Q128JVS, Package_SO:SOIC-8_5.23x5.23mm_P1.27mm, symbol Memory_Flash:W25Q128JVS
- added U3: MCP2515-xSO, Package_SO:SOIC-18W_7.5x11.6mm_P1.27mm, symbol Interface_CAN_LIN:MCP2515-xSO
- added U4: TJA1042T3118, Package_SO:HTSOP-8-1EP_3.9x4.9mm_P1.27mm_EP2.4x3.2mm, symbol OpenEFI-STM32-rev3:TJA1042T3118
- added U5: TPD2E2U06, Package_TO_SOT_SMD:SOT-143, symbol Power_Protection:TPD2E2U06
- added Y2: 12MHz, Crystal:Crystal_SMD_3225-4Pin_3.2x2.5mm, symbol Device:Crystal_GND24
- C1, C5, C6: value 100nF -> 30pF; footprint Capacitor_SMD:C_0805_2012Metric -> Capacitor_SMD:C_0603_1608Metric; LCSC C49678 -> (none)
- C10, C22, C8: footprint Capacitor_SMD:C_0805_2012Metric -> Capacitor_SMD:C_0603_1608Metric; LCSC C49678 -> (none)
- C11, C12: value 2.2uF -> 100nF; footprint Capacitor_SMD:C_0805_2012Metric -> Capacitor_SMD:C_0603_1608Metric; LCSC C49217 -> (none); Note Low ESR <2Ohm -> (none)
- C14, C15: value 15pF -> 100nF; footprint Capacitor_SMD:C_0805_2012Metric -> Capacitor_SMD:C_0603_1608Metric; LCSC C1794 -> (none)
- C2: value 1uF -> 30pF; footprint Capacitor_SMD:C_0805_2012Metric -> Capacitor_SMD:C_0603_1608Metric; LCSC C28323 -> (none)
- C20: value 4.7nF -> 100nF; footprint Capacitor_SMD:C_0805_2012Metric -> Capacitor_SMD:C_0603_1608Metric; LCSC C77475 -> (none)
- C3, C4, C7: value 100nF -> 2.2uF; footprint Capacitor_SMD:C_0805_2012Metric -> Capacitor_SMD:C_0603_1608Metric; LCSC C49678 -> (none)
- Y1: value 25MHz -> 8MHz; LCSC (none) -> C9002
Connections:
- net GND1 is gone; now on net GND: C22.2, J1.4 (GND), J1.5 (Shield)
- net NRST is gone; now on net GND: C10.2
- net d+ is gone; now on net USB_D+: J1.3 (D+)
- net d- is gone; now on net USB_D-: J1.2 (D-)
- net +3V3: now also C10.1, C11.1, C12.1, C14.1, C15.1, C20.1, C22.1, C3.2, C7.2, C8.2, J2.1 (Pin_1), R13.2, R14.2, U1.1 (IOVDD), U1.10 (IOVDD), U1.22 (IOVDD), U1.26 (RUN), U1.33 (IOVDD), U1.42 (IOVDD), U1.44 (VREG_IN), U1.48 (USB_VDD), U1.49 (IOVDD), U2.8 (VCC), U3.18 (VDD), U4.5 (VIO); no longer C1.1, C2.1, C3.1, C4.1, C5.1, C6.1, C7.1, C8.1
- net +5V: now also BATT_CONN1.1 (Pin_1), DISPLAY1.1 (Pin_1), FUEL_CONN1.1 (Pin_1), O2_CONN1.1 (Pin_1), OIL_CONN1.1 (Pin_1), OIL_TEMP1.1 (Pin_1), RPM_CONN1.1 (Pin_1), SPEED_CONN1.1 (Pin_1), TEMP1.1 (Pin_1), U4.3 (VCC)
- net CAN+: now also J3.4 (Pin_4), J4.4 (Pin_4), R15.2, U4.7 (CANH)
- net CAN-: now also J3.3 (Pin_3), J4.3 (Pin_3), R16.2, U4.6 (CANL)
- net GND: now also C1.1, C2.1, C3.1, C4.1, C5.1, C6.1, C7.1, C8.1, BATT_CONN1.8 (Pin_8), C26.2, C27.2, C28.2, C9.2, DISPLAY1.8 (Pin_8), FUEL_CONN1.8 (Pin_8), J2.5 (Pin_5), J3.1 (Pin_1), J4.1 (Pin_1), JP2.1 (A), O2_CONN1.8 (Pin_8), OIL_CONN1.8 (Pin_8), OIL_TEMP1.8 (Pin_8), R17.1, R18.1, R19.1, RPM_CONN1.8 (Pin_8), SPEED_CONN1.8 (Pin_8), TEMP1.8 (Pin_8), U1.19 (TESTEN), U1.57 (GND), U2.4 (GND), U3.9 (VSS), U4.2 (GND), U4.8 (STB), U5.1 (GND), Y2.1, Y2.3; no longer C1.2, C10.1, C2.2, C3.2, C4.2, C5.2, C6.2, C7.2, C8.2
- net I2C1_SCL: now also U1.13 (GPIO10)
- net I2C1_SDA: now also U1.12 (GPIO9)
- net PWM_BACK_1: now also U10.17 (LED10); no longer U10.13 (LED7)
- net PWM_BACK_2: now also U10.18 (LED11); no longer U10.15 (LED8)
- net PWM_BAR1: now also U10.11 (LED5); no longer U10.8 (LED2)
- net PWM_BAR2: now also U10.12 (LED6); no longer U10.9 (LED3)
- net PWM_BAR3: now also U10.13 (LED7); no longer U10.10 (LED4)
- net PWM_FUEL1: now also U10.9 (LED3); no longer U10.6 (LED0)
- net PWM_FUEL2: now also U10.10 (LED4); no longer U10.7 (LED1)
- net PWM_OD: now also U10.16 (LED9); no longer U10.12 (LED6)
- net PWM_VEL: now also U10.15 (LED8); no longer U10.11 (LED5)
- net SYS_SWCLK: now also J2.4 (Pin_4), U1.24 (SWCLK)
- net SYS_SWDIO: now also J2.2 (Pin_2), U1.25 (SWD)
- net USB_D+: now also R2.1, U5.2
- net USB_D-: now also R1.2, U5.3
- net at J1.1 (VBUS): now also U5.4 (VBUS); no longer C22.1
- net OSC_IN renamed CAN_CLOCK_B
- net CAN_CLOCK_B: now also C2.2, U3.7 (OSC2); no longer C14.1
- net OSC_OUT renamed CAN_CLOCK_A
- net CAN_CLOCK_A: now also C1.2, U3.8 (OSC1); no longer C15.1
- net SPI2_MISO renamed SPI_MISO
- net SPI2_MOSI renamed SPI_MOSI
- net SPI2_SCK renamed SPI_SCK
- new net: R1.1, U1.46 (USB_DM)
- new net: C9.1, R15.1, R16.1
- new net: JP2.2 (B), R3.2
- new net: U3.1 (TXCAN), U4.4 (RXD)
- new net: R13.1, U3.17 (~{RESET})
- new net: U3.2 (RXCAN), U4.1 (TXD)
- new net: D4.1 (K), R17.2
- new net: R14.1, R3.1, U1.56 (QSPI_SS), U2.1 (~{CS})
- new net: R2.2, U1.47 (USB_DP)
- new net: U1.51 (QSPI_SD3), U2.7 (IO3)
- new net: U1.52 (QSPI_SCLK), U2.6 (CLK)
- new net: U1.53 (QSPI_SD0), U2.5 (DI(IO0))
- new net: U1.54 (QSPI_SD2), U2.3 (IO2)
- new net: U1.55 (QSPI_SD1), U2.2 (DO(IO1))
- new net: D6.1 (K), R19.2
- new net: D5.1 (K), R18.2
- new net +1V1: C27.1, C4.2, U1.23 (DVDD), U1.45 (VREG_VOUT), U1.50 (DVDD)
- new net BATT_CS: BATT_CONN1.5 (Pin_5)
- new net CF_CONF0: U1.16 (GPIO13)
- new net CF_CONF1: U1.17 (GPIO14)
- new net CF_CONF2: U1.18 (GPIO15)
- new net CLK: BATT_CONN1.2 (Pin_2), DISPLAY1.2 (Pin_2), FUEL_CONN1.2 (Pin_2), O2_CONN1.2 (Pin_2), OIL_CONN1.2 (Pin_2), OIL_TEMP1.2 (Pin_2), RPM_CONN1.2 (Pin_2), SPEED_CONN1.2 (Pin_2), TEMP1.2 (Pin_2), U1.30 (GPIO19)
- new net DISPLAY_CS: DISPLAY1.5 (Pin_5)
- new net FUEL_CS: FUEL_CONN1.5 (Pin_5)
- new net GPIO0: U1.2 (GPIO0), U3.13 (SCK)
- new net GPIO1: U1.3 (GPIO1), U3.14 (SI)
- new net GPIO2: U1.4 (GPIO2), U3.15 (SO)
- new net GPIO3: U1.5 (GPIO3)
- new net GPIO4: U1.6 (GPIO4)
- new net GPIO5: U1.7 (GPIO5)
- new net GPIO6: U1.8 (GPIO6)
- new net GPIO7: U1.9 (GPIO7)
- new net GPIO8: U1.11 (GPIO8), U3.16 (~{CS})
- new net Ip_dac: U1.36 (GPIO24)
- new net Ip_sense: U1.40 (GPIO28_ADC2)
- new net LED_BLUE: D5.2 (A), U1.28 (GPIO17)
- new net LED_GREEN: D4.2 (A), U1.27 (GPIO16)
- new net LED_RED: D6.2 (A), U1.29 (GPIO18)
- new net LSU_Vm: U1.35 (GPIO23)
- new net MISO: BATT_CONN1.3 (Pin_3), DISPLAY1.3 (Pin_3), FUEL_CONN1.3 (Pin_3), O2_CONN1.3 (Pin_3), OIL_CONN1.3 (Pin_3), OIL_TEMP1.3 (Pin_3), RPM_CONN1.3 (Pin_3), SPEED_CONN1.3 (Pin_3), TEMP1.3 (Pin_3), U1.31 (GPIO20)
- new net MOSI: BATT_CONN1.4 (Pin_4), DISPLAY1.4 (Pin_4), FUEL_CONN1.4 (Pin_4), O2_CONN1.4 (Pin_4), OIL_CONN1.4 (Pin_4), OIL_TEMP1.4 (Pin_4), RPM_CONN1.4 (Pin_4), SPEED_CONN1.4 (Pin_4), TEMP1.4 (Pin_4), U1.32 (GPIO21)
- new net O2_CS: O2_CONN1.5 (Pin_5)
- new net OIL_CS: OIL_CONN1.5 (Pin_5)
- new net OIL_TEMP_CS: OIL_TEMP1.5 (Pin_5)
- new net PWM_BACK_BATT: BATT_CONN1.6 (Pin_6)
- new net PWM_BACK_DISPLAY: DISPLAY1.6 (Pin_6)
- new net PWM_BACK_O2: O2_CONN1.6 (Pin_6)
- new net PWM_BACK_OIL: OIL_CONN1.6 (Pin_6)
- new net PWM_BACK_OIL_TEMP: OIL_TEMP1.6 (Pin_6)
- new net PWM_BACK_RPM: FUEL_CONN1.6 (Pin_6), RPM_CONN1.6 (Pin_6), U10.6 (LED0)
- new net PWM_BACK_TEMP: TEMP1.6 (Pin_6)
- new net PWM_SPEED1: SPEED_CONN1.6 (Pin_6), U10.7 (LED1)
- new net PWM_SPEED2: SPEED_CONN1.7 (Pin_7), U10.8 (LED2)
- new net RPM_CS: RPM_CONN1.5 (Pin_5)
- new net SPEED_CS: SPEED_CONN1.5 (Pin_5)
- new net TEMP_CS: TEMP1.5 (Pin_5)
- new net UN_SENSE: U1.41 (GPIO29_ADC3)
- new net VDDA: C26.1, U1.43 (ADC_AVDD)
- new net Vm: U1.39 (GPIO27_ADC1)
- new net xin: C5.2, U1.20 (XIN), Y2.2
- new net xout: C6.2, U1.21 (XOUT), Y2.4
- no-connect marks 7 -> 26
Other:
- note added: "ADC & USB"
- note added: "CAN CONNECTOR (FTCAN Compatible)"
- note added: "CAN Clock"
- note added: "DVDD DECOUPLING"
- note added: "IOVDD DECOUPLING"
- note removed: "Crystal"
- note removed: "DEBUG PIN"
- note removed: "USB Protection (Optional)"
- note removed: "VDD Decoupling"
- note removed: "VREF Decoupling"
- moved on the sheet: C16, C17, C18, C19, U10, U11, U9

Commit message: ESD SPI
Parts:
- added C23, C24, C29, C30, C31, C32, C33: 100nF, Capacitor_SMD:C_0603_1608Metric, symbol Device:C_Small
- added U12, U14, U15, U16, U17, U6, U8: SRV05-4, Package_TO_SOT_SMD:SOT-23-6, symbol Power_Protection:SRV05-4
Connections:
- net Ip_dac is gone; now on net I2C1_SDA: U1.36 (GPIO24)
- net LSU_Vm is gone; now on net I2C1_SCL: U1.35 (GPIO23)
- net +3V3: now also C23.2, C24.2, C29.2, C30.2, C31.2, C32.2, C33.2, U12.5 (VP), U14.5 (VP), U15.5 (VP), U16.5 (VP), U17.5 (VP), U6.5 (VP), U8.5 (VP)
- net BATT_CS: now also U8.1 (IO1)
- net CLK: now also U6.1 (IO1)
- net DISPLAY_CS: now also U6.6 (IO4)
- net FUEL_CS: now also U16.4 (IO3)
- net GND: now also C23.1, C24.1, C29.1, C30.1, C31.1, C32.1, C33.1, U12.2 (VN), U14.2 (VN), U15.2 (VN), U16.2 (VN), U17.2 (VN), U6.2 (VN), U8.2 (VN)
- net I2C1_SCL: no longer U1.13 (GPIO10)
- net I2C1_SDA: no longer U1.12 (GPIO9)
- net MISO: now also U6.3 (IO2)
- net MOSI: now also U6.4 (IO3)
- net O2_CS: now also U16.6 (IO4)
- net OIL_CS: now also U8.4 (IO3)
- net OIL_TEMP_CS: now also U8.3 (IO2)
- net PWM_BACK_BATT: now also U14.1 (IO1), U17.1 (IO1)
- net PWM_BACK_DISPLAY: now also U15.1 (IO1)
- net PWM_BACK_O2: now also U15.4 (IO3)
- net PWM_BACK_OIL: now also U15.3 (IO2)
- net PWM_BACK_OIL_TEMP: now also U14.3 (IO2), U17.3 (IO2)
- net PWM_BACK_RPM: now also U12.1 (IO1); no longer FUEL_CONN1.6 (Pin_6)
- net PWM_BACK_TEMP: now also U15.6 (IO4)
- net PWM_SPEED1: now also U12.4 (IO3)
- net PWM_SPEED2: now also U12.6 (IO4)
- net RPM_CS: now also U16.1 (IO1)
- net SPEED_CS: now also U16.3 (IO2)
- net TEMP_CS: now also U8.6 (IO4)
- net MOSI2: now reaches U1.14 (GPIO11)
- net MOSI2: now also U3.15 (SO)
- net CS_CAN: now reaches U1.15 (GPIO12)
- net CS_CAN: now also U3.16 (~{CS})
- net CF_CONF0: no longer names the net of U1.16 (GPIO13)
- net CF_CONF1: no longer names the net of U1.17 (GPIO14)
- net CF_CONF2: no longer names the net of U1.18 (GPIO15)
- net GPIO0: no longer names the net of U1.2 (GPIO0)
- net GPIO0: no longer U3.13 (SCK)
- net GPIO1: no longer names the net of U1.3 (GPIO1)
- net GPIO1: no longer U3.14 (SI)
- net GPIO2: no longer names the net of U1.4 (GPIO2)
- net GPIO2: no longer U3.15 (SO)
- net GPIO3: no longer names the net of U1.5 (GPIO3)
- net GPIO4: no longer names the net of U1.6 (GPIO4)
- net GPIO5: no longer names the net of U1.7 (GPIO5)
- net GPIO6: no longer names the net of U1.8 (GPIO6)
- net GPIO7: no longer names the net of U1.9 (GPIO7)
- net GPIO8: no longer names the net of U1.11 (GPIO8)
- net GPIO8: no longer U3.16 (~{CS})
- net Ip_sense: no longer names the net of U1.40 (GPIO28_ADC2)
- net UN_SENSE: no longer names the net of U1.41 (GPIO29_ADC3)
- net Vm: no longer names the net of U1.39 (GPIO27_ADC1)
- new net CLK2: U1.12 (GPIO9), U3.13 (SCK)
- new net MISO2: U1.13 (GPIO10), U3.14 (SI)
- new net PWM_BACK_FUEL: U12.3 (IO2)
- new net PWM_BACK_FUEl: FUEL_CONN1.6 (Pin_6)
- no-connect marks 26 -> 25
Other:
- note added: "ESD"
- moved on the sheet: BATT_CONN1, C21, C25, C3, C4, C7, C8, C9, D1, D2, D3, DISPLAY1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

Commit message: add powaaaaaa
Parts:
- added D? (x2): 1N5822, Diode_THT:D_DO-201AD_P15.24mm_Horizontal, symbol Diode:1N5822
- added U?: GL2576-3.3TA5R, Package_TO_SOT_SMD:TO-263-5_TabPin3, symbol Regulator_Switching:GL2576-3.3TA5R
- added U?: GL2576-5.0TA5R, Package_TO_SOT_SMD:TO-263-5_TabPin3, symbol Regulator_Switching:GL2576-5.0TA5R
Other:
- moved on the sheet: C3, C4, C7, C8, JP2, R1, R14, R2, R3, U1, U2
