File: pcb/v2/dashdashv2/dashdashv2.kicad_sch (KiCad schematic)
At the start: 95 parts, among them J1 USB_B, J10 O2_CONN1, J11 BATT_CONN1, J12 OIL_CONN1, J13 OIL_TEMP1, J2 Tag connect, J3 Conn_01x04_Female, J4 Conn_01x04_Female, J5 SPEED_CONN1, J6 DISPLAY1, J7 RPM_CONN1, J8 TEMP1, J9 FUEL_CONN1, Q1 IRF540N, Q2 IRF540N, Q3 2N3904, U1 RP2040, U10 PCA9685PW, U11 MIC2940A-3.3WU, U12 SRV05-4, U13 LT4363IMS, U14 SRV05-4, U15 SRV05-4, U16 SRV05-4, U17 SRV05-4, U19 GL2576-5.0TA5R, U2 W25Q128JVS, U3 MCP2515-xSO, U4 TJA1042T3118, U5 TPD2E2U06, U6 SRV05-4, U7 25LCxxx, U8 SRV05-4, U9 MIC2940A-5.0WT, Y1 8MHz, Y2 12MHz

Commit message: routing can/usb/power/leds/flash
Parts:
- removed C1, C2: 30pF, Capacitor_SMD:C_0603_1608Metric, symbol Device:C_Small
- removed C13: 100nF, Capacitor_SMD:C_0805_2012Metric, symbol Device:C_Small
- removed C16, C17, C18, C19: CP_Small, symbol Device:CP_Small
- removed C21: 47nF, Capacitor_SMD:C_0603_1608Metric, symbol Device:C_Small
- removed C23, C24, C29, C30, C31, C32, C33: 100nF, Capacitor_SMD:C_0603_1608Metric, symbol Device:C_Small
- removed C25: 0.1uF, Capacitor_SMD:C_0603_1608Metric, symbol Device:C_Small
- removed C3: 2.2uF, Capacitor_SMD:C_0603_1608Metric, symbol Device:C_Small
- removed C9: 4.7nF, Capacitor_SMD:C_0805_2012Metric, symbol Device:C_Small
- removed D1: SMAJ58CA, Diode_SMD:D_SMA, symbol Device:D_TVS
- removed D2, D3: 1N4148, Diode_SMD:D_0805_2012Metric, symbol Diode:1N4148
- removed D7: 1N5822, Diode_THT:D_DO-201AD_P15.24mm_Horizontal, symbol Diode:1N5822
- removed J10: O2_CONN1, Connector_PinHeader_1.27mm:PinHeader_2x05_P1.27mm_Vertical, symbol Connector_Generic:Conn_02x05_Odd_Even
- removed J11: BATT_CONN1, Connector_PinHeader_1.27mm:PinHeader_2x05_P1.27mm_Vertical, symbol Connector_Generic:Conn_02x05_Odd_Even
- removed J12: OIL_CONN1, Connector_PinHeader_1.27mm:PinHeader_2x05_P1.27mm_Vertical, symbol Connector_Generic:Conn_02x05_Odd_Even
- removed J13: OIL_TEMP1, Connector_PinHeader_1.27mm:PinHeader_2x05_P1.27mm_Vertical, symbol Connector_Generic:Conn_02x05_Odd_Even
- removed J3, J4: Conn_01x04_Female, Connector_Molex:Molex_Mini-Fit_Jr_5569-04A1_2x02_P4.20mm_Horizontal, symbol Connector:Conn_01x04_Female
- removed J5: SPEED_CONN1, Connector_PinHeader_1.27mm:PinHeader_2x05_P1.27mm_Vertical, symbol Connector_Generic:Conn_02x05_Odd_Even
- removed J6: DISPLAY1, Connector_PinHeader_1.27mm:PinHeader_2x05_P1.27mm_Vertical, symbol Connector_Generic:Conn_02x05_Odd_Even
- removed J7: RPM_CONN1, Connector_PinHeader_1.27mm:PinHeader_2x05_P1.27mm_Vertical, symbol Connector_Generic:Conn_02x05_Odd_Even
- removed J8: TEMP1, Connector_PinHeader_1.27mm:PinHeader_2x05_P1.27mm_Vertical, symbol Connector_Generic:Conn_02x05_Odd_Even
- removed J9: FUEL_CONN1, Connector_PinHeader_1.27mm:PinHeader_2x05_P1.27mm_Vertical, symbol Connector_Generic:Conn_02x05_Odd_Even
- removed JP1: Jumper_NO_Small, Jumper:SolderJumper-2_P1.3mm_Open_TrianglePad1.0x1.5mm, symbol Device:Jumper_NO_Small
- removed Q1, Q2: IRF540N, Package_TO_SOT_THT:TO-220-3_Vertical, symbol Transistor_FET:IRF540N
- removed Q3: 2N3904, Package_TO_SOT_SMD:TSOT-23, symbol Transistor_BJT:2N3904
- removed R12: 10K 1/10W, Resistor_SMD:R_0603_1608Metric, symbol Device:R_Small
- removed R13: 10k, Resistor_SMD:R_0603_1608Metric, symbol Device:R
- removed R15, R16: 30R, Resistor_SMD:R_1206_3216Metric, symbol Device:R_Small
- removed R4: 0.01R, Resistor_SMD:R_1210_3225Metric, symbol Device:R_Small
- removed R5: 57.6K 1/10W, Resistor_SMD:R_0603_1608Metric, symbol Device:R_Small
- removed R6: 4.99K 1/10W, Resistor_SMD:R_0603_1608Metric, symbol Device:R_Small
- removed R7, R8: 10R 1/10W, Resistor_SMD:R_0603_1608Metric, symbol Device:R_Small
- removed R9: 1M 1/10W, Resistor_SMD:R_0603_1608Metric, symbol Device:R_Small
- removed U11: MIC2940A-3.3WU, Package_TO_SOT_SMD:TO-263-3_TabPin2, symbol Regulator_Linear:L7805
- removed U12, U14, U15, U16, U17, U6, U8: SRV05-4, Package_TO_SOT_SMD:SOT-23-6, symbol Power_Protection:SRV05-4
- removed U13: LT4363IMS, Package_SO:SOIC-16W_7.5x10.3mm_P1.27mm, symbol OpenEFI-STM32-rev3:LT4363IMS
- removed U19: GL2576-5.0TA5R, Package_TO_SOT_SMD:TO-263-5_TabPin3, symbol Regulator_Switching:GL2576-5.0TA5R
- removed U3: MCP2515-xSO, Package_SO:SOIC-18W_7.5x11.6mm_P1.27mm, symbol Interface_CAN_LIN:MCP2515-xSO
- removed U4: TJA1042T3118, Package_SO:HTSOP-8-1EP_3.9x4.9mm_P1.27mm_EP2.4x3.2mm, symbol OpenEFI-STM32-rev3:TJA1042T3118
- removed U7: 25LCxxx, Package_SO:SOIC-8_3.9x4.9mm_P1.27mm, symbol Memory_EEPROM:25LCxxx
- removed U9: MIC2940A-5.0WT, Package_TO_SOT_THT:TO-220-3_Vertical, symbol Regulator_Linear:L7805
- removed Y1: 8MHz, Crystal:Crystal_SMD_3225-4Pin_3.2x2.5mm, symbol Device:Crystal_GND24
- added D2: D_Zener, Diode_SMD:D_SOD-123F, symbol Device:D_Zener
- added H1, H2, H3, H4, H5: MountingHole, MountingHole:MountingHole_2.2mm_M2_Pad_Via, symbol Mechanical:MountingHole
- added R10: 5k, Resistor_SMD:R_0603_1608Metric, symbol Device:R
- added R11: 1k, Resistor_SMD:R_0603_1608Metric, symbol Device:R
- J2: footprint Connector:Tag-Connect_TC2030-IDC-NL_2x03_P1.27mm_Vertical -> Connector:Tag-Connect_TC2030-IDC-FP_2x03_P1.27mm_Vertical
Connections:
- net PWM_BAR1 is gone; now on net PWM_BACK_OIL: U10.11 (LED5)
- net PWM_BAR2 is gone; now on net PWM_BACK_O2: U10.12 (LED6)
- net PWM_BAR3 is gone; now on net PWM_BACK_TEMP: U10.13 (LED7)
- net PWM_FUEL1 is gone; now on net PWM_SPEED2: U10.9 (LED3)
- net PWM_FUEL2 is gone; now on net PWM_BACK_DISPLAY: U10.10 (LED4)
- net PWM_OD is gone; now on net PWM_BACK_OIL_TEMP: U10.16 (LED9)
- net PWM_VEL is gone; now on net PWM_BACK_BATT: U10.15 (LED8)
- net +12V: now also R10.1
- net +1V1: now also C28.1
- net +3V3: no longer C7.2, C8.2
- net BATT_CS: now also U1.7 (GPIO5)
- net CLK2: now also U1.15 (GPIO12); no longer U1.12 (GPIO9)
- net CS_CAN: now also U1.12 (GPIO9); no longer U1.15 (GPIO12)
- net DISPLAY_CS: now also U1.8 (GPIO6)
- net FUEL_CS: now also U1.3 (GPIO1)
- net GND: now also C8.2, D2.2 (A), R11.2; no longer C8.1
- net I2C1_SCL: now also U10.26 (SCL); no longer U10.27 (SDA)
- net I2C1_SDA: now also U10.27 (SDA); no longer U10.26 (SCL)
- net MISO2: now also U1.14 (GPIO11); no longer U1.13 (GPIO10)
- net MOSI2: now also U1.13 (GPIO10); no longer U1.14 (GPIO11)
- net O2_CS: now also U1.5 (GPIO3)
- net OIL_CS: now also U1.6 (GPIO4)
- net OIL_TEMP_CS: now also U1.11 (GPIO8)
- net PWM_BACK_FUEL: now also U10.7 (LED1)
- net PWM_SPEED1: now also U10.8 (LED2); no longer U10.7 (LED1)
- net PWM_SPEED2: no longer U10.8 (LED2)
- net RPM_CS: now also U1.2 (GPIO0)
- net SPEED_CS: now also U1.4 (GPIO2)
- net TEMP_CS: now also U1.9 (GPIO7)
- net D+: now reaches R1.1, U1.46 (USB_DM)
- net QSPI_SS: now reaches R14.1, R3.1, U1.56 (QSPI_SS), U2.1 (~{CS})
- net 12V_ACC: now reaches U1.17 (GPIO14)
- net 12V_LIGHT: now reaches U1.18 (GPIO15)
- net 12V_ENABLE: now reaches U1.37 (GPIO25)
- net at U1.38 (GPIO26_ADC0): now also D2.1 (K), R10.2, R11.1
- net ENCODER_A: now reaches U1.39 (GPIO27_ADC1)
- net ENCODER_B: now reaches U1.40 (GPIO28_ADC2)
- net ENCODER_C: now reaches U1.41 (GPIO29_ADC3)
- net D-: now reaches R2.2, U1.47 (USB_DP)
- net QSPI_SD3: now reaches U1.51 (QSPI_SD3), U2.7 (IO3)
- net QSPI_SCLK: now reaches U1.52 (QSPI_SCLK), U2.6 (CLK)
- net QSPI_SD0: now reaches U1.53 (QSPI_SD0), U2.5 (DI(IO0))
- net QSPI_SD2: now reaches U1.54 (QSPI_SD2), U2.3 (IO2)
- net QSPI_SD1: now reaches U1.55 (QSPI_SD1), U2.2 (DO(IO1))
- net PWM_BACK_1: no longer names the net of U10.17 (LED10)
- net PWM_BACK_2: no longer names the net of U10.18 (LED11)
- new net: C7.2, C8.1
- no-connect marks 25 -> 11
Other:
- added sheet CAN (can.kicad_sch)
- added sheet Connectors (connectors.kicad_sch)
- added sheet ESD (esd.kicad_sch)
- added sheet Power (power.kicad_sch)
- note removed: "CAN"
- note removed: "CAN CONNECTOR (FTCAN Compatible)"
- note removed: "CAN Clock"
- note removed: "ESD"
- note removed: "Surge Protection (optional)"
- note removed: "UNLIMITED POWAAAAA"
- moved on the sheet: C10, C11, C12, C14, C15, C20, C22, C26, C27, C28, C4, C7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

Commit message: routing
Parts:
- removed C14: 100nF, Capacitor_SMD:C_0603_1608Metric, symbol Device:C_Small
Connections:
- net +3V3: now also C7.2, C8.1
- net CLK: now also U1.27 (GPIO16); no longer U1.30 (GPIO19)
- net LED_BLUE: now also U1.31 (GPIO20); no longer U1.28 (GPIO17)
- net LED_GREEN: now also U1.30 (GPIO19); no longer U1.27 (GPIO16)
- net LED_RED: now also U1.32 (GPIO21); no longer U1.29 (GPIO18)
- net MISO: now also U1.28 (GPIO17); no longer U1.31 (GPIO20)
- net MOSI: now also U1.29 (GPIO18); no longer U1.32 (GPIO21)
- net PWM_BACK_FUEL renamed PWM_BACK_FUEl
Changed lines of the file:
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@@
   (junction (at 217.17 62.865) (diameter 0.9144) (color 0 0 0 0)
+  )
+  (junction (at 130.81 166.37) (diameter 0) (color 0 0 0 0)
   )
   (junction (at 41.275 177.8) (diameter 0) (color 0 0 0 0)
@@
     (stroke (width 0) (type default) (color 0 0 0 0))
   )
+  (wire (pts (xy 130.81 166.37) (xy 133.985 166.37))
+    (stroke (width 0) (type default) (color 0 0 0 0))
+  )
   (wire (pts (xy 154.94 76.2) (xy 156.845 76.2))
     (stroke (width 0) (type default) (color 0 0 0 0))
@@
     (stroke (width 0) (type solid) (color 0 0 0 0))
   )
+  (wire (pts (xy 130.81 166.37) (xy 130.81 168.91))
+    (stroke (width 0) (type default) (color 0 0 0 0))
+  )
   (wire (pts (xy 127 45.72) (xy 127 43.18))
     (stroke (width 0) (type default) (color 0 0 0 0))
@@
   )
   (wire (pts (xy 15.24 45.085) (xy 26.67 45.085))
-    (stroke (width 0) (type default) (color 0 0 0 0))
-  )
-  (wire (pts (xy 127.635 166.37) (xy 133.985 166.37))
     (stroke (width 0) (type default) (color 0 0 0 0))
   )
@@
     (stroke (width 0) (type solid) (color 0 0 0 0))
   )
-  (wire (pts (xy 130.81 165.1) (xy 130.81 168.91))
+  (wire (pts (xy 130.81 165.1) (xy 130.81 166.37))
     (stroke (width 0) (type default) (color 0 0 0 0))
   )
@@
   )
   (wire (pts (xy 88.9 106.68) (xy 91.44 106.68))
+    (stroke (width 0) (type default) (color 0 0 0 0))
+  )
+  (wire (pts (xy 127.635 166.37) (xy 130.81 166.37))
     (stroke (width 0) (type default) (color 0 0 0 0))
   )
@@
     (effects (font (size 1.27 1.27)) (justify left bottom))
   )
-  (label "LED_RED" (at 88.9 109.22 180)
+  (label "LED_RED" (at 88.9 116.84 180)
     (effects (font (size 1.27 1.27)) (justify right bottom))
   )
@@
     (effects (font (size 1.27 1.27)) (justify left bottom))
   )
-  (label "LED_BLUE" (at 88.9 106.68 180)
+  (label "LED_BLUE" (at 88.9 114.3 180)
     (effects (font (size 1.27 1.27)) (justify right bottom))
   )
@@
     (effects (font (size 1.27 1.27)) (justify left bottom))
   )
-  (label "LED_GREEN" (at 88.9 104.14 180)
+  (label "LED_GREEN" (at 88.9 111.76 180)
     (effects (font (size 1.27 1.27)) (justify right bottom))
   )
@@
     )
   )
-  (global_label "PWM_BACK_FUEL" (shape input) (at 261.62 29.845 0) (fields_autoplaced)
-    (effects (font (size 0.8 0.8)) (justify left))
-    (property "Referencias entre hojas" "${INTERSHEET_REFS}" (id 0) (at 272.9686 29.895 0)
-      (effects (font (size 0.8 0.8)) (justify left) hide)
-    )
-  )
   (global_label "12V_LIGHT" (shape input) (at 78.105 101.6 180) (fields_autoplaced)
     (effects (font (size 1 1)) (justify right))
@@
     )
   )
+  (global_label "PWM_BACK_FUEl" (shape input) (at 261.62 29.845 0) (fields_autoplaced)
+    (effects (font (size 0.9 0.9)) (justify left))
+    (property "Referencias entre hojas" "${INTERSHEET_REFS}" (id 0) (at 274.13 29.7888 0)
+      (effects (font (size 0.9 0.9)) (justify left) hide)
+    )
+  )
   (global_label "TEMP_CS" (shape input) (at 85.725 81.28 180) (fields_autoplaced)
     (effects (font (size 1.27 1.27)) (justify right))
@@
     )
   )
-  (global_label "MOSI" (shape input) (at 88.9 116.84 180) (fields_autoplaced)
+  (global_label "MOSI" (shape input) (at 88.9 109.22 180) (fields_autoplaced)
     (effects (font (size 1.27 1.27)) (justify right))
-    (property "Referencias entre hojas" "${INTERSHEET_REFS}" (id 0) (at 81.8907 116.7606 0)
+    (property "Referencias entre hojas" "${INTERSHEET_REFS}" (id 0) (at 81.8907 109.1406 0)
       (effects (font (size 1.27 1.27)) (justify right) hide)
     )
@@
     )
   )
-  (global_label "CLK" (shape input) (at 88.9 111.76 180) (fields_autoplaced)
+  (global_label "CLK" (shape input) (at 88.9 104.14 180) (fields_autoplaced)
     (effects (font (size 1.27 1.27)) (justify right))
-    (property "Referencias entre hojas" "${INTERSHEET_REFS}" (id 0) (at 82.9188 111.6806 0)
+    (property "Referencias entre hojas" "${INTERSHEET_REFS}" (id 0) (at 82.9188 104.0606 0)
       (effects (font (size 1.27 1.27)) (justify right) hide)
     )
   )
-  (global_label "MISO" (shape input) (at 88.9 114.3 180) (fields_autoplaced)
+  (global_label "MISO" (shape input) (at 88.9 106.68 180) (fields_autoplaced)
     (effects (font (size 1.27 1.27)) (justify right))
-    (property "Referencias entre hojas" "${INTERSHEET_REFS}" (id 0) (at 81.8907 114.2206 0)
+    (property "Referencias entre hojas" "${INTERSHEET_REFS}" (id 0) (at 81.8907 106.6006 0)
       (effects (font (size 1.27 1.27)) (justify right) hide)
     )
@@
     (pin "2")
   )
-  (symbol (lib_id "Device:C_Small") (at 46.355 182.88 0) (unit 1)
-    (in_bom yes) (on_board yes)
-    (property "Reference" "C14" (id 0) (at 46.355 180.34 0)
-      (effects (font (size 1.27 1.27)) (justify left))
-    )
-    (property "Value" "100nF" (id 1) (at 48.6791 184.5885 0)
-      (effects (font (size 1.27 1.27)) (justify left) hide)
-    )
-    (property "Footprint" "Capacitor_SMD:C_0603_1608Metric" (id 2) (at 46.355 182.88 0)
-      (effects (font (size 1.27 1.27)) hide)
-    )
-    (property "Datasheet" "~" (id 3) (at 46.355 182.88 0)
-      (effects (font (size 1.27 1.27)) hide)
-    )
-    (pin "1")
-    (pin "2")
-  )
   (symbol (lib_id "power:GND") (at 73.66 154.305 0) (unit 1)
     (in_bom yes) (on_board yes) (fields_autoplaced)
@@
       (reference "C12") (unit 1) (value "100nF") (footprint "Capacitor_SMD:C_0603_1608Metric")
     )
-    (path "/9f5ee244-2191-40d3-9edc-28834d3b8ffb"
-      (reference "C14") (unit 1) (value "100nF") (footprint "Capacitor_SMD:C_0603_1608Metric")
-    )
     (path "/c84f2060-c609-4a66-ba37-90b6184c19dd"
