File: pcb/v2/dashdashv2/tachometer/rev2/tach.kicad_sch (KiCad schematic)
At the start: 87 parts

Commit message: update neopixel
Parts:
- D1, D10, D11, D111, D112, D113, D114, D115, D12, D13, D14, D15, D16, D17, D18, D19, D2, D20, D21, D22, D23, D24, D25, D26, D27, D28, D29, D3, D30, D31, D32, D33, D34, D35, D36, D37, D38, D39, D4, D40, D41, D5, D6, D7, D8, D9: footprint LED_SMD:LED_Cree-PLCC4_2x2mm_CW -> dashdash_lib:LED_WS2812-2020; symbol LED:WS2812B -> LED:SK6812MINI
Connections:
- net +5VA: now also D1.4 (VDD), D10.4 (VDD), D11.4 (VDD), D111.4 (VDD), D112.4 (VDD), D113.4 (VDD), D114.4 (VDD), D115.4 (VDD), D12.4 (VDD), D13.4 (VDD), D14.4 (VDD), D15.4 (VDD), D16.4 (VDD), D17.4 (VDD), D18.4 (VDD), D19.4 (VDD), D2.4 (VDD), D20.4 (VDD), D21.4 (VDD), D22.4 (VDD), D23.4 (VDD), D24.4 (VDD), D25.4 (VDD), D26.4 (VDD), D27.4 (VDD), D28.4 (VDD), D29.4 (VDD), D3.4 (VDD), D30.4 (VDD), D31.4 (VDD), D32.4 (VDD), D33.4 (VDD), D34.4 (VDD), D35.4 (VDD), D36.4 (VDD), D37.4 (VDD), D38.4 (VDD), D39.4 (VDD), D4.4 (VDD), D40.4 (VDD), D41.4 (VDD), D5.4 (VDD), D6.4 (VDD), D7.4 (VDD), D8.4 (VDD), D9.4 (VDD); no longer D1.1 (VDD), D10.1 (VDD), D11.1 (VDD), D111.1 (VDD), D112.1 (VDD), D113.1 (VDD), D114.1 (VDD), D115.1 (VDD), D12.1 (VDD), D13.1 (VDD), D14.1 (VDD), D15.1 (VDD), D16.1 (VDD), D17.1 (VDD), D18.1 (VDD), D19.1 (VDD), D2.1 (VDD), D20.1 (VDD), D21.1 (VDD), D22.1 (VDD), D23.1 (VDD), D24.1 (VDD), D25.1 (VDD), D26.1 (VDD), D27.1 (VDD), D28.1 (VDD), D29.1 (VDD), D3.1 (VDD), D30.1 (VDD), D31.1 (VDD), D32.1 (VDD), D33.1 (VDD), D34.1 (VDD), D35.1 (VDD), D36.1 (VDD), D37.1 (VDD), D38.1 (VDD), D39.1 (VDD), D4.1 (VDD), D40.1 (VDD), D41.1 (VDD), D5.1 (VDD), D6.1 (VDD), D7.1 (VDD), D8.1 (VDD), D9.1 (VDD)
- net DIN: now also D1.3 (DIN); no longer D1.4 (DIN)
- net GND: now also D1.2 (VSS), D10.2 (VSS), D11.2 (VSS), D111.2 (VSS), D112.2 (VSS), D113.2 (VSS), D114.2 (VSS), D115.2 (VSS), D12.2 (VSS), D13.2 (VSS), D14.2 (VSS), D15.2 (VSS), D16.2 (VSS), D17.2 (VSS), D18.2 (VSS), D19.2 (VSS), D2.2 (VSS), D20.2 (VSS), D21.2 (VSS), D22.2 (VSS), D23.2 (VSS), D24.2 (VSS), D25.2 (VSS), D26.2 (VSS), D27.2 (VSS), D28.2 (VSS), D29.2 (VSS), D3.2 (VSS), D30.2 (VSS), D31.2 (VSS), D32.2 (VSS), D33.2 (VSS), D34.2 (VSS), D35.2 (VSS), D36.2 (VSS), D37.2 (VSS), D38.2 (VSS), D39.2 (VSS), D4.2 (VSS), D40.2 (VSS), D41.2 (VSS), D5.2 (VSS), D6.2 (VSS), D7.2 (VSS), D8.2 (VSS), D9.2 (VSS); no longer D1.3 (VSS), D10.3 (VSS), D11.3 (VSS), D111.3 (VSS), D112.3 (VSS), D113.3 (VSS), D114.3 (VSS), D115.3 (VSS), D12.3 (VSS), D13.3 (VSS), D14.3 (VSS), D15.3 (VSS), D16.3 (VSS), D17.3 (VSS), D18.3 (VSS), D19.3 (VSS), D2.3 (VSS), D20.3 (VSS), D21.3 (VSS), D22.3 (VSS), D23.3 (VSS), D24.3 (VSS), D25.3 (VSS), D26.3 (VSS), D27.3 (VSS), D28.3 (VSS), D29.3 (VSS), D3.3 (VSS), D30.3 (VSS), D31.3 (VSS), D32.3 (VSS), D33.3 (VSS), D34.3 (VSS), D35.3 (VSS), D36.3 (VSS), D37.3 (VSS), D38.3 (VSS), D39.3 (VSS), D4.3 (VSS), D40.3 (VSS), D41.3 (VSS), D5.3 (VSS), D6.3 (VSS), D7.3 (VSS), D8.3 (VSS), D9.3 (VSS)
- new net: D2.1 (DOUT), D3.3 (DIN)
- new net: D1.1 (DOUT), D111.3 (DIN), D2.3 (DIN)
- new net: D16.1 (DOUT), D17.3 (DIN)
- new net: D15.1 (DOUT), D16.3 (DIN)
- new net: D114.1 (DOUT), D115.3 (DIN)
- new net: D6.1 (DOUT), D7.3 (DIN)
- new net: D5.1 (DOUT), D6.3 (DIN)
- new net: D29.1 (DOUT), D30.3 (DIN)
- new net: D28.1 (DOUT), D29.3 (DIN)
- new net: D4.1 (DOUT), D5.3 (DIN)
- new net: D35.1 (DOUT), D36.3 (DIN)
- new net: D34.1 (DOUT), D35.3 (DIN)
- new net: D32.1 (DOUT), D33.3 (DIN)
- new net: D31.1 (DOUT), D32.3 (DIN)
- new net: D23.1 (DOUT), D24.3 (DIN)
- new net: D22.1 (DOUT), D23.3 (DIN)
- new net: D112.1 (DOUT), D113.3 (DIN)
- new net: D111.1 (DOUT), D112.3 (DIN)
- new net: D11.1 (DOUT), D12.3 (DIN)
- new net: D10.1 (DOUT), D11.3 (DIN)
- new net: D13.1 (DOUT), D14.3 (DIN)
- new net: D12.1 (DOUT), D13.3 (DIN)
- new net: D20.1 (DOUT), D21.3 (DIN)
- new net: D19.1 (DOUT), D20.3 (DIN)
- new net: D113.1 (DOUT), D114.3 (DIN)
- new net: D33.1 (DOUT), D34.3 (DIN)
- new net: D30.1 (DOUT), D31.3 (DIN)
- new net: D17.1 (DOUT), D18.3 (DIN)
- new net: D18.1 (DOUT), D19.3 (DIN)
- new net: D14.1 (DOUT), D15.3 (DIN)
- new net: D24.1 (DOUT), D25.3 (DIN)
- new net: D21.1 (DOUT), D22.3 (DIN)
- new net: D3.1 (DOUT), D4.3 (DIN)
- new net: D37.1 (DOUT), D38.3 (DIN)
- new net: D36.1 (DOUT), D37.3 (DIN)
- new net: D40.1 (DOUT), D41.3 (DIN)
- new net: D39.1 (DOUT), D40.3 (DIN)
- new net: D7.1 (DOUT), D8.3 (DIN)
- new net: D10.3 (DIN), D9.1 (DOUT)
- new net: D8.1 (DOUT), D9.3 (DIN)
- new net: D38.1 (DOUT), D39.3 (DIN)
- new net: D27.1 (DOUT), D28.3 (DIN)
- new net: D26.1 (DOUT), D27.3 (DIN)
- new net: D25.1 (DOUT), D26.3 (DIN)
